File: augertapowermanagementv3.kicad_pcb (KiCad board)
At the start: 4 copper layers, 316.7 x 183 mm, 82 parts, among them J1 Screw_Terminal_01x02, J10 Screw_Terminal_01x10, J11 Screw_Terminal_01x10, J12 gnd block, J2 76825-0002, J3 USB_A_Stacked, J4 USB_A_Stacked, J5 USB_A_Stacked, J6 USB_A_Stacked, J7 Screw_Terminal_01x08, J8 Screw_Terminal_01x10, J9 5v block, K1 J107F1CS203VDC.80, K2 J107F1CS203VDC.80, SW1 SW_SPDT, U1 LM2596_5v, U10 INA219AxD, U11 INA219AxD, U12 LM2596_5v, U13 LM2596_5v, U14 INA219AxD, U15 INA219AxD, U16 LM2596_11.5v, U17 LM2596_5v, U18 INA219AxD, U19 INA219AxD, U2 ESP32-DEVKITC-32D, U20 LM2596_11.5v, U21 INA219AxD, U22 LM2596_11.5v, U23 INA219AxD, U24 MCP9808_MSOP, U3 INA219AxD, U4 LM2596_5v, U5 LM2596_5v, U6 INA219AxD, U7 INA219AxD, U8 LM2596_5v, U9 LM2596_5v

Commit message: updates v4
Routing:
- net /power_conversion/pi 5v: track 0.00 -> 814.8 mm, vias 0 -> 13
- net /power_conversion/SDA: track 0.00 -> 673.6 mm, vias 0 -> 12
- net /power_conversion/SCL: track 0.00 -> 662.1 mm, vias 0 -> 11
- net -BATT: track 0.00 -> 292.8 mm, vias 0 -> 21
- net Net-(C2-Pad1): track 0.00 -> 283.4 mm
- net Net-(F1-Pad2): track 0.00 -> 253.3 mm, vias 0 -> 1
- net /power_conversion/N1: track 0.00 -> 194.9 mm, vias 0 -> 1
- net /power_conversion/spare2: track 0.00 -> 181.0 mm
- net /power_conversion/N3: track 0.00 -> 147.8 mm, vias 0 -> 2
- net Net-(JP5-Pad2): track 0.00 -> 144.9 mm, vias 0 -> 1
- net /power_conversion/battery+: track 0.00 -> 142.2 mm, vias 0 -> 2
- net /power_conversion/N4: track 0.00 -> 135.7 mm
- net /power_conversion/N2: track 0.00 -> 134.9 mm, vias 0 -> 2
- net /power_conversion/pi1: track 0.00 -> 108.1 mm, vias 0 -> 2
- net Net-(J11-Pad3): track 0.00 -> 103.9 mm
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- added copper zone on In2.Cu, net +BATT
- added copper zone on B.Cu, net -BATT
- added copper zone on In2.Cu, net Net-(F1-Pad2)
- removed copper zone on In1.Cu, net +BATT
- removed copper zone on In2.Cu, net -BATT
