File: power_conversion.kicad_sch (KiCad schematic)
At the start: 54 parts, among them U10 INA219AxD, U11 INA219AxD, U12 LM2596_5v, U13 LM2596_5v, U14 INA219AxD, U15 INA219AxD, U16 LM2596_11.5v, U17 LM2596_5v, U18 INA219AxD, U19 INA219AxD, U20 LM2596_11.5v, U21 INA219AxD, U22 LM2596_11.5v, U23 INA219AxD, U3 INA219AxD, U4 LM2596_5v, U5 LM2596_5v, U6 INA219AxD, U7 INA219AxD, U8 LM2596_5v, U9 LM2596_5v

Commit message: updated
Parts:
- C1: Purchase (none) -> https://www.digikey.com/en/products/detail/kemet/CDR33BX104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
- F1, F2: Purchase (none) -> https://www.digikey.com/en/products/detail/littelfuse-inc/1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
- JP2, JP3, JP4, JP6: Purchase (none) -> NA, JUST pads
- R10, R11, R14, R15, R3, R4, R5, R6, R7, R8, R9: Purchase (none) -> https://www.digikey.com/en/products/detail/rohm-semiconduct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
- R12, R13: Purchase (none) -> https://www.digikey.com/en/products/detail/yageo/RT2512FKE0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
- U10, U11, U14, U15, U18, U19, U21, U23, U3, U6, U7: Purchase (none) -> https://www.digikey.com/en/products/detail/texas-instrument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
- U12, U13, U17, U4, U5, U8, U9: Purchase (none) -> https://www.amazon.com/LM2596-Converter-Module-Supply-1-23V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

Commit message: update
Parts:
- TP10, TP11, TP12, TP13, TP14, TP15, TP16, TP17, TP18, TP6, TP7, TP8, TP9: Purchase (none) -> JUST PAD
- U16, U20, U22: Purchase (none) -> IN LAB
Changed lines of the file:
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@@
+      (effects (font (size 1.27 1.27)) hide)
+    )
+    (property "Purchase" "JUST PAD" (id 4) (at 86.36 116.84 0)
       (effects (font (size 1.27 1.27)) hide)
     )
@@
       (effects (font (size 1.27 1.27)) hide)
     )
+    (property "Purchase" "JUST PAD" (id 4) (at 228.6 80.01 0)
+      (effects (font (size 1.27 1.27)) hide)
+    )
     (pin "1")
   )
@@
       (effects (font (size 1.27 1.27)) hide)
     )
+    (property "Purchase" "JUST PAD" (id 4) (at 21.59 33.02 0)
+      (effects (font (size 1.27 1.27)) hide)
+    )
     (pin "1")
   )
@@
     )
     (property "Datasheet" "~" (id 3) (at 231.14 102.87 0)
+      (effects (font (size 1.27 1.27)) hide)
+    )
+    (property "Purchase" "JUST PAD" (id 4) (at 226.06 102.87 0)
       (effects (font (size 1.27 1.27)) hide)
     )
@@
       (effects (font (size 1.27 1.27)) hide)
     )
+    (property "Purchase" "JUST PAD" (id 4) (at 227.33 50.8 0)
+      (effects (font (size 1.27 1.27)) hide)
+    )
     (pin "1")
   )
@@
     )
     (property "Datasheet" "" (id 3) (at 64.77 172.72 0)
+      (effects (font (size 1.27 1.27)) hide)
+    )
+    (property "Purchase" "IN LAB" (id 4) (at 66.04 172.72 0)
       (effects (font (size 1.27 1.27)) hide)
     )
@@
       (effects (font (size 1.27 1.27)) hide)
     )
+    (property "Purchase" "JUST PAD" (id 4) (at 199.39 26.67 0)
+      (effects (font (size 1.27 1.27)) hide)
+    )
     (pin "1")
   )
@@
     )
     (property "Datasheet" "~" (id 3) (at 44.45 33.02 0)
+      (effects (font (size 1.27 1.27)) hide)
+    )
+    (property "Purchase" "JUST PAD" (id 4) (at 39.37 33.02 0)
       (effects (font (size 1.27 1.27)) hide)
     )
@@
       (effects (font (size 1.27 1.27)) hide)
     )
+    (property "Purchase" "JUST PAD" (id 4) (at 85.09 49.53 0)
+      (effects (font (size 1.27 1.27)) hide)
+    )
     (pin "1")
   )
@@
       (effects (font (size 1.27 1.27)) hide)
     )
+    (property "Purchase" "IN LAB" (id 4) (at 66.04 147.32 0)
+      (effects (font (size 1.27 1.27)) hide)
+    )
     (pin "1")
     (pin "2")
@@
       (effects (font (size 1.27 1.27)) hide)
     )
+    (property "Purchase" "JUST PAD" (id 4) (at 85.09 144.78 0)
+      (effects (font (size 1.27 1.27)) hide)
+    )
     (pin "1")
   )
@@
     )
     (property "Datasheet" "~" (id 3) (at 237.49 132.08 0)
+      (effects (font (size 1.27 1.27)) hide)
+    )
+    (property "Purchase" "JUST PAD" (id 4) (at 232.41 132.08 0)
       (effects (font (size 1.27 1.27)) hide)
     )
@@
       (effects (font (size 1.27 1.27)) hide)
     )
+    (property "Purchase" "JUST PAD" (id 4) (at 81.28 170.18 0)
+      (effects (font (size 1.27 1.27)) hide)
+    )
     (pin "1")
   )
@@
     )
     (property "Datasheet" "~" (id 3) (at 88.9 92.71 0)
+      (effects (font (size 1.27 1.27)) hide)
+    )
+    (property "Purchase" "JUST PAD" (id 4) (at 83.82 92.71 0)
       (effects (font (size 1.27 1.27)) hide)
     )
@@
       (effects (font (size 1.27 1.27)) hide)
     )
+    (property "Purchase" "IN LAB" (id 4) (at 66.04 120.65 0)
+      (effects (font (size 1.27 1.27)) hide)
+    )
     (pin "1")
     (pin "2")
@@
       (effects (font (size 1.27 1.27)) hide)
     )
+    (property "Purchase" "JUST PAD" (id 4) (at 83.82 72.39 0)
+      (effects (font (size 1.27 1.27)) hide)
+    )

Commit message: update
Parts:
- JP2, JP6: footprint Connector_PinHeader_2.00mm:PinHeader_1x02_P2.00mm_Horizontal -> cit:JUMPER_5102TR; Purchase NA, JUST pads -> https://www.digikey.com/en/products/detail/keystone-electro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
Changed lines of the file:
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@@
       (effects (font (size 1.27 1.27)) (justify right))
     )
-    (property "Footprint" "Connector_PinHeader_2.00mm:PinHeader_1x02_P2.00mm_Horizontal" (id 2) (at 34.29 35.56 0)
-      (effects (font (size 1.27 1.27)) hide)
-    )
-    (property "Datasheet" "~" (id 3) (at 34.29 35.56 0)
-      (effects (font (size 1.27 1.27)) hide)
-    )
-    (property "Purchase" "NA, JUST pads" (id 4) (at 34.29 35.56 0)
+    (property "Footprint" "cit:JUMPER_5102TR" (id 2) (at 34.29 35.56 0)
+      (effects (font (size 1.27 1.27)) hide)
+    )
+    (property "Datasheet" "https://www.digikey.com/en/products/detail/keystone-electronics/5102TR/4759688" (id 3) (at 34.29 35.56 0)
+      (effects (font (size 1.27 1.27)) hide)
+    )
+    (property "Purchase" "https://www.digikey.com/en/products/detail/keystone-electronics/5102TR/4759688" (id 4) (at 34.29 35.56 0)
       (effects (font (size 1.27 1.27)) hide)
     )
@@
     (property "Reference" "JP2" (id 0) (at 27.94 21.59 0))
     (property "Value" "Jumper_2_Open" (id 1) (at 27.94 24.13 0))
-    (property "Footprint" "Connector_PinHeader_2.00mm:PinHeader_1x02_P2.00mm_Horizontal" (id 2) (at 27.94 27.94 0)
-      (effects (font (size 1.27 1.27)) hide)
-    )
-    (property "Datasheet" "~" (id 3) (at 27.94 27.94 0)
-      (effects (font (size 1.27 1.27)) hide)
-    )
-    (property "Purchase" "NA, JUST pads" (id 4) (at 27.94 27.94 0)
-      (effects (font (size 1.27 1.27)) hide)
-    )
+    (property "Footprint" "cit:JUMPER_5102TR" (id 2) (at 27.94 27.94 0)
+      (effects (font (size 1.27 1.27)) hide)
+    )
+    (property "Datasheet" "https://www.digikey.com/en/products/detail/keystone-electronics/5102TR/4759688" (id 3) (at 27.94 27.94 0)
+      (effects (font (size 1.27 1.27)) hide)
+    )
+    (property "Purchase" "https://www.digikey.com/en/products/detail/keystone-electronics/5102TR/4759688" (id 4) (at 27.94 27.94 0)
+      (effects (font (size 1.27 1.27)) hide)
+    )

Commit message: Improved power plane, relay changes, i2c resistor changes
Parts:
- R12, R13: value 3.3K -> 5k; footprint Resistor_SMD:R_2512_6332Metric_Pad1.40x3.35mm_HandSolder -> Resistor_SMD:R_1206_3216Metric_Pad1.30x1.75mm_HandSolder; Purchase https://www.digikey.com/en/products/detail/yageo/RT2512FKE0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 -> https://www.digikey.com/en/products/detail/yageo/RT1206BRD0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
Connections:
- net Buck in: now reaches F1.2, F2.2, JP3.2 (B), JP4.2 (B), JP6.1 (A), R3.2, TP6.1, U12.1 (Vin), U13.1 (Vin), U16.1 (Vin), U17.1 (Vin), U3.8 (IN+), U4.1 (Vin), U5.1 (Vin), U8.1 (Vin), U9.1 (Vin)
- net pi 5v renamed 3v3
Changed lines of the file:
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@@
     (effects (font (size 1.27 1.27)) (justify left bottom))
   )
+  (label "Buck in" (at 46.99 58.42 0)
+    (effects (font (size 1.27 1.27)) (justify left bottom))
+  )
   (hierarchical_label "SDA" (shape bidirectional) (at 119.38 151.13 0)
     (effects (font (size 1.27 1.27)) (justify left))
@@
     (effects (font (size 1.27 1.27)) (justify left))
   )
-  (hierarchical_label "pi 5v" (shape input) (at 148.59 185.42 270)
+  (hierarchical_label "3v3" (shape input) (at 148.59 185.42 270)
     (effects (font (size 1.27 1.27)) (justify right))
   )
@@
     (effects (font (size 1.27 1.27)) (justify left))
   )
-  (hierarchical_label "pi 5v" (shape input) (at 143.51 83.82 0)
+  (hierarchical_label "3v3" (shape input) (at 143.51 83.82 0)
     (effects (font (size 1.27 1.27)) (justify left))
   )
@@
     (effects (font (size 1.27 1.27)) (justify right))
   )
-  (hierarchical_label "pi 5v" (shape input) (at 260.35 124.46 90)
-    (effects (font (size 1.27 1.27)) (justify left))
-  )
-  (hierarchical_label "pi 5v" (shape input) (at 119.38 161.29 270)
+  (hierarchical_label "3v3" (shape input) (at 260.35 124.46 90)
+    (effects (font (size 1.27 1.27)) (justify left))
+  )
+  (hierarchical_label "3v3" (shape input) (at 119.38 161.29 270)
     (effects (font (size 1.27 1.27)) (justify right))
   )
@@
     (effects (font (size 1.27 1.27)) (justify right))
   )
-  (hierarchical_label "pi 5v" (shape input) (at 115.57 93.98 90)
+  (hierarchical_label "3v3" (shape input) (at 115.57 93.98 90)
     (effects (font (size 1.27 1.27)) (justify left))
   )
@@
     (effects (font (size 1.27 1.27)) (justify right))
   )
-  (hierarchical_label "pi 5v" (shape input) (at 135.89 119.38 90)
+  (hierarchical_label "3v3" (shape input) (at 135.89 119.38 90)
     (effects (font (size 1.27 1.27)) (justify left))
   )
@@
     (effects (font (size 1.27 1.27)) (justify right))
   )
-  (hierarchical_label "pi 5v" (shape input) (at 116.84 50.8 90)
+  (hierarchical_label "3v3" (shape input) (at 116.84 50.8 90)
     (effects (font (size 1.27 1.27)) (justify left))
   )
@@
     (effects (font (size 1.27 1.27)) (justify left))
   )
-  (hierarchical_label "pi 5v" (shape input) (at 193.04 132.08 90)
-    (effects (font (size 1.27 1.27)) (justify left))
-  )
-  (hierarchical_label "pi 5v" (shape input) (at 109.22 146.05 90)
+  (hierarchical_label "3v3" (shape input) (at 193.04 132.08 90)
+    (effects (font (size 1.27 1.27)) (justify left))
+  )
+  (hierarchical_label "3v3" (shape input) (at 109.22 146.05 90)
     (effects (font (size 1.27 1.27)) (justify left))
   )
@@
     (effects (font (size 1.27 1.27)) (justify right))
   )
-  (hierarchical_label "pi 5v" (shape input) (at 229.87 19.05 90)
+  (hierarchical_label "3v3" (shape input) (at 229.87 19.05 90)
     (effects (font (size 1.27 1.27)) (justify left))
   )
@@
     (effects (font (size 1.27 1.27)) (justify left))
   )
-  (hierarchical_label "pi 5v" (shape input) (at 246.38 50.8 90)
+  (hierarchical_label "3v3" (shape input) (at 246.38 50.8 90)
     (effects (font (size 1.27 1.27)) (justify left))
   )
@@
     (effects (font (size 1.27 1.27)) (justify left))
   )
-  (hierarchical_label "pi 5v" (shape input) (at 254 107.95 0)
+  (hierarchical_label "3v3" (shape input) (at 254 107.95 0)
     (effects (font (size 1.27 1.27)) (justify left))
   )
@@
     (effects (font (size 1.27 1.27)) (justify left))
   )
-  (hierarchical_label "pi 5v" (shape input) (at 256.54 66.04 270)
+  (hierarchical_label "3v3" (shape input) (at 256.54 66.04 270)
     (effects (font (size 1.27 1.27)) (justify right))
   )
@@
     (effects (font (size 1.27 1.27)) (justify left))
   )
-  (hierarchical_label "pi 5v" (shape input) (at 243.84 95.25 90)
-    (effects (font (size 1.27 1.27)) (justify left))
-  )
-  (hierarchical_label "pi 5v" (shape input) (at 240.03 34.29 270)
+  (hierarchical_label "3v3" (shape input) (at 243.84 95.25 90)
+    (effects (font (size 1.27 1.27)) (justify left))
+  )
+  (hierarchical_label "3v3" (shape input) (at 240.03 34.29 270)
     (effects (font (size 1.27 1.27)) (justify right))
   )
@@
     (effects (font (size 1.27 1.27)) (justify left))
   )
-  (hierarchical_label "pi 5v" (shape input) (at 138.43 170.18 90)
+  (hierarchical_label "3v3" (shape input) (at 138.43 170.18 90)
     (effects (font (size 1.27 1.27)) (justify left))
   )
@@
     (effects (font (size 1.27 1.27)) (justify left))
   )
-  (hierarchical_label "pi 5v" (shape input) (at 166.37 132.08 90)
-    (effects (font (size 1.27 1.27)) (justify left))
-  )
-  (hierarchical_label "pi 5v" (shape input) (at 133.35 71.12 90)
-    (effects (font (size 1.27 1.27)) (justify left))
-  )
-  (hierarchical_label "pi 5v" (shape input) (at 262.89 72.39 90)
-    (effects (font (size 1.27 1.27)) (justify left))
-  )
-  (hierarchical_label "pi 5v" (shape input) (at 179.07 132.08 90)
+  (hierarchical_label "3v3" (shape input) (at 166.37 132.08 90)
+    (effects (font (size 1.27 1.27)) (justify left))
+  )
+  (hierarchical_label "3v3" (shape input) (at 133.35 71.12 90)
+    (effects (font (size 1.27 1.27)) (justify left))
+  )
+  (hierarchical_label "3v3" (shape input) (at 262.89 72.39 90)
+    (effects (font (size 1.27 1.27)) (justify left))
+  )
+  (hierarchical_label "3v3" (shape input) (at 179.07 132.08 90)
     (effects (font (size 1.27 1.27)) (justify left))
   )
@@
       (effects (font (size 1.27 1.27)) (justify left))
     )
-    (property "Value" "3.3K" (id 1) (at 168.91 137.1599 0)
-      (effects (font (size 1.27 1.27)) (justify left))
-    )
-    (property "Footprint" "Resistor_SMD:R_2512_6332Metric_Pad1.40x3.35mm_HandSolder" (id 2) (at 167.386 136.144 90)
+    (property "Value" "5k" (id 1) (at 168.91 137.1599 0)
+      (effects (font (size 1.27 1.27)) (justify left))
+    )
+    (property "Footprint" "Resistor_SMD:R_1206_3216Metric_Pad1.30x1.75mm_HandSolder" (id 2) (at 167.386 136.144 90)
       (effects (font (size 1.27 1.27)) hide)
     )
@@
       (effects (font (size 1.27 1.27)) hide)
     )
-    (property "Purchase" "https://www.digikey.com/en/products/detail/yageo/RT2512FKE073K3L/5947596" (id 4) (at 166.37 135.89 0)
+    (property "Purchase" "https://www.digikey.com/en/products/detail/yageo/RT1206BRD075KL/5936961" (id 4) (at 166.37 135.89 0)
       (effects (font (size 1.27 1.27)) hide)
     )
@@
       (effects (font (size 1.27 1.27)) (justify left))
     )
-    (property "Value" "3.3K" (id 1) (at 181.61 137.1599 0)
-      (effects (font (size 1.27 1.27)) (justify left))
-    )
-    (property "Footprint" "Resistor_SMD:R_2512_6332Metric_Pad1.40x3.35mm_HandSolder" (id 2) (at 180.086 136.144 90)
+    (property "Value" "5k" (id 1) (at 181.61 137.1599 0)
+      (effects (font (size 1.27 1.27)) (justify left))
+    )
+    (property "Footprint" "Resistor_SMD:R_1206_3216Metric_Pad1.30x1.75mm_HandSolder" (id 2) (at 180.086 136.144 90)
       (effects (font (size 1.27 1.27)) hide)
     )
@@
       (effects (font (size 1.27 1.27)) hide)
     )
-    (property "Purchase" "https://www.digikey.com/en/products/detail/yageo/RT2512FKE073K3L/5947596" (id 4) (at 179.07 135.89 0)
-      (effects (font (size 1.27 1.27)) hide)
-    )
+    (property "Purchase" "https://www.digikey.com/en/products/detail/yageo/RT1206BRD075KL/5936961" (id 4) (at 179.07 135.89 0)
+      (effects (font (size 1.27 1.27)) hide)
+    )
