File: power_conversion.kicad_sch (KiCad schematic)
At the start: 59 parts, among them U10 INA219AxD, U11 INA219AxD, U12 LM2596_5v, U13 LM2596_5v, U14 INA219AxD, U15 INA219AxD, U16 LM2596_11.5v, U17 LM2596_5v, U18 INA219AxD, U19 INA219AxD, U20 LM2596_11.5v, U21 INA219AxD, U22 LM2596_11.5v, U23 INA219AxD, U3 INA219AxD, U4 LM2596_5v, U5 LM2596_5v, U6 INA219AxD, U7 INA219AxD, U8 LM2596_5v, U9 LM2596_5v

Commit message: updates
Parts:
- removed F? (x11): Polyfuse, symbol Device:Polyfuse
Connections:
- net battery+: now also R3.2, TP6.1, U13.1 (Vin), U16.1 (Vin), U17.1 (Vin), U3.8 (IN+), U4.1 (Vin), U5.1 (Vin), U8.1 (Vin), U9.1 (Vin)
- net at JP4.1 (A): now also U22.1 (Vin)
- net at JP3.1 (A): now also U20.1 (Vin)

Commit message: 04/13/2023
Parts:
- removed C1: 0.1uF, Capacitor_SMD:C_1210_3225Metric_Pad1.33x2.70mm_HandSolder, symbol Device:C
- removed R12, R13: 5k, Resistor_SMD:R_1206_3216Metric_Pad1.30x1.75mm_HandSolder, symbol Device:R_US
- removed U12, U13, U17, U4, U5, U8, U9: LM2596_5v, lm2596:DC_DC_LM2596_small, symbol powermanagement:YAAJ_DCDC_StepDown_LM2596
- removed U16, U20, U22: LM2596_11.5v, lm2596:DC_DC_LM2596_small, symbol powermanagement:YAAJ_DCDC_StepDown_LM2596
Connections:
- net Regulator (5V, 3A)/V­­_out: now reaches R10.2, TP15.1, U18.8 (IN+)
- net Regulator (5V, 3A)5/V­­_out: now reaches R7.2, TP12.1, U11.8 (IN+)
- net Regulator (5V, 3A)2/V­­_out: now reaches R6.2, TP11.1, U10.8 (IN+)
- net Regulator (5V, 3A)6/V­­_out: now reaches R9.2, TP14.1, U15.8 (IN+)
- net Regulator (5V, 3A)4/V­­_out: now reaches R5.2, TP10.1, U7.8 (IN+)
- net Regulator (Adjustable, 3A)1/V_in: now reaches JP4.1 (A)
- net Regulator (Adjustable, 3A)1/V_out: now reaches R15.2, TP18.1, U23.8 (IN+)
- net Regulator (5V, 3A)7/V­­_out: now reaches R11.2, TP16.1, U19.8 (IN+)
- net Regulator (Adjustable, 3A)/V_out: now reaches R14.2, TP17.1, U21.8 (IN+)
- net Regulator (Adjustable, 3A)/V_in: now reaches JP3.1 (A)
- net Regulator (5V, 3A)1/V­­_out: now reaches R4.2, TP9.1, U6.8 (IN+)
- net Regulator (5V, 3A)1/V­­_out: now reaches R8.2, TP13.1, U14.8 (IN+)
Other:
- added sheet Regulator (5V, 3A) (test.kicad_sch)
- added sheet Regulator (5V, 3A)1 (test.kicad_sch)
- added sheet Regulator (5V, 3A)2 (test.kicad_sch)
- added sheet Regulator (5V, 3A)4 (test.kicad_sch)
- added sheet Regulator (5V, 3A)5 (test.kicad_sch)
- added sheet Regulator (5V, 3A)6 (test.kicad_sch)
- added sheet Regulator (5V, 3A)7 (test.kicad_sch)
- added sheet Regulator (Adjustable, 3A) (Adjustable Regulator.kicad_sch)
- added sheet Regulator (Adjustable, 3A)1 (Adjustable Regulator.kicad_sch)

Commit message: hi
Connections:
- net Regulator (5V, 3A)/V­­_out renamed Regulator (Adjustable, 3A)2/V_out
- net Regulator (5V, 3A)1/V­­_out renamed Regulator (Adjustable, 3A)5/V_out
- net Regulator (5V, 3A)1/V­­_out renamed Regulator (Adjustable, 3A)3/V_out
- net Regulator (5V, 3A)2/V­­_out renamed Regulator (Adjustable, 3A)4/V_out
- net Regulator (5V, 3A)4/V­­_out renamed Regulator (Adjustable, 3A)6/V_out
- net Regulator (5V, 3A)5/V­­_out renamed Regulator (Adjustable, 3A)7/V_out
- net Regulator (5V, 3A)6/V­­_out renamed Regulator (Adjustable, 3A)8/V_out
- net Regulator (5V, 3A)7/V­­_out renamed Regulator (Adjustable, 3A)9/V_out
Other:
- removed sheet Regulator (5V, 3A)
- removed sheet Regulator (5V, 3A)1
- removed sheet Regulator (5V, 3A)2
- removed sheet Regulator (5V, 3A)4
- removed sheet Regulator (5V, 3A)5
- removed sheet Regulator (5V, 3A)6
- removed sheet Regulator (5V, 3A)7
- added sheet Regulator (Adjustable, 3A)2 (Adjustable Regulator.kicad_sch)
- added sheet Regulator (Adjustable, 3A)3 (Adjustable Regulator.kicad_sch)
- added sheet Regulator (Adjustable, 3A)4 (Adjustable Regulator.kicad_sch)
- added sheet Regulator (Adjustable, 3A)5 (Adjustable Regulator.kicad_sch)
- added sheet Regulator (Adjustable, 3A)6 (Adjustable Regulator.kicad_sch)
- added sheet Regulator (Adjustable, 3A)7 (Adjustable Regulator.kicad_sch)
- added sheet Regulator (Adjustable, 3A)8 (Adjustable Regulator.kicad_sch)
- added sheet Regulator (Adjustable, 3A)9 (Adjustable Regulator.kicad_sch)

Commit message: finish assigning componets
Parts:
- added C14: 680u, Capacitor_THT:CP_Radial_D35.0mm_P10.00mm_SnapIn, symbol Device:C
- renumbered R9 to R10, R5 to R11, R11 to R12, R7 to R13, R14 to R3, R8 to R4, R4 to R5, R10 to R7, R15 to R8, R3 to R9, TP6 to TP10, TP14 to TP11, TP10 to TP12, TP12 to TP13, TP16 to TP14, TP18 to TP4, TP11 to TP5, TP13 to TP6, TP9 to TP7, TP17 to TP8, TP15 to TP9, U15 to U10, U7 to U11, U19 to U12, U11 to U13, U21 to U3, U14 to U4, U6 to U5, U10 to U6, U18 to U7, U23 to U8, U3 to U9
Connections:
- net GND: now also C14.2
- net battery+: now also C14.1

Commit message: fix lot of errors
Parts:
- added R47, R48: 2.2k, Resistor_SMD:R_1210_3225Metric_Pad1.30x2.65mm_HandSolder, symbol Device:R_US
Connections:
- net 3v3: now also R47.1, R48.1
- net SCL: now also R47.2
- net SDA: now also R48.2
Changed lines of the file:
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@@
   (junction (at 227.33 50.8) (diameter 0) (color 0 0 0 0)
   )
+  (junction (at 173.99 88.9) (diameter 0) (color 0 0 0 0)
+  )
   (junction (at 48.26 72.39) (diameter 0) (color 0 0 0 0)
   )
@@
     (stroke (width 0) (type default))
   )
+  (wire (pts (xy 173.99 88.9) (xy 170.18 88.9))
+    (stroke (width 0) (type default))
+  )
   (wire (pts (xy 236.22 50.8) (xy 227.33 50.8))
     (stroke (width 0) (type default))
@@
     (stroke (width 0) (type default))
   )
+  (wire (pts (xy 173.99 78.74) (xy 173.99 88.9))
+    (stroke (width 0) (type default))
+  )
   (wire (pts (xy 186.69 38.1) (xy 120.65 38.1))
     (stroke (width 0) (type default))
@@
     (stroke (width 0) (type default))
   )
+  (wire (pts (xy 180.34 88.9) (xy 173.99 88.9))
+    (stroke (width 0) (type default))
+  )
   (wire (pts (xy 119.38 158.75) (xy 124.46 158.75))
     (stroke (width 0) (type default))
@@
     (stroke (width 0) (type default))
   )
+  (wire (pts (xy 170.18 96.52) (xy 170.18 100.33))
+    (stroke (width 0) (type default))
+  )
   (wire (pts (xy 148.59 182.88) (xy 148.59 185.42))
     (stroke (width 0) (type default))
@@
   )
   (wire (pts (xy 48.26 170.18) (xy 55.88 170.18))
+    (stroke (width 0) (type default))
+  )
+  (wire (pts (xy 180.34 96.52) (xy 180.34 100.33))
     (stroke (width 0) (type default))
   )
@@
     (effects (font (size 1.27 1.27)) (justify left))
   )
+  (hierarchical_label "SDA" (shape bidirectional) (at 180.34 100.33 270) (fields_autoplaced)
+    (effects (font (size 1.27 1.27)) (justify right))
+  )
   (hierarchical_label "3v3" (shape input) (at 135.89 119.38 90) (fields_autoplaced)
     (effects (font (size 1.27 1.27)) (justify left))
@@
     (effects (font (size 1.27 1.27)) (justify right))
   )
+  (hierarchical_label "SCL" (shape bidirectional) (at 170.18 100.33 270) (fields_autoplaced)
+    (effects (font (size 1.27 1.27)) (justify right))
+  )
   (hierarchical_label "SCL" (shape bidirectional) (at 146.05 132.08 0) (fields_autoplaced)
     (effects (font (size 1.27 1.27)) (justify left))
@@
   (hierarchical_label "SDA" (shape bidirectional) (at 270.51 139.7 270) (fields_autoplaced)
     (effects (font (size 1.27 1.27)) (justify right))
+  )
+  (hierarchical_label "3v3" (shape input) (at 173.99 78.74 90) (fields_autoplaced)
+    (effects (font (size 1.27 1.27)) (justify left))
   )
   (hierarchical_label "SCL" (shape bidirectional) (at 119.38 153.67 0) (fields_autoplaced)
@@
         (path "/65134029-dbd2-409a-85a8-13c2a33ff019/8a8c373f-9bc3-4cf7-8f41-4802da916698"
           (reference "R6") (unit 1)
+        )
+      )
+    )
+  )
+  (symbol (lib_id "Device:R_US") (at 180.34 92.71 0) (unit 1)
+    (in_bom yes) (on_board yes) (dnp no) (fields_autoplaced)
+    (property "Reference" "R48" (at 182.88 92.075 0)
+      (effects (font (size 1.27 1.27)) (justify left))
+    )
+    (property "Value" "2.2k" (at 182.88 94.615 0)
+      (effects (font (size 1.27 1.27)) (justify left))
+    )
+    (property "Footprint" "Resistor_SMD:R_1210_3225Metric_Pad1.30x2.65mm_HandSolder" (at 181.356 92.964 90)
+      (effects (font (size 1.27 1.27)) hide)
+    )
+    (property "Datasheet" "~" (at 180.34 92.71 0)
+      (effects (font (size 1.27 1.27)) hide)
+    )
+    (pin "1")
+    (pin "2")
+    (instances
+      (project "augertapowermanagement"
+        (path "/65134029-dbd2-409a-85a8-13c2a33ff019/8a8c373f-9bc3-4cf7-8f41-4802da916698"
+          (reference "R48") (unit 1)
         )
       )
@@
         )
       )
+    )
+  )
+  (symbol (lib_id "Device:R_US") (at 170.18 92.71 0) (unit 1)
+    (in_bom yes) (on_board yes) (dnp no) (fields_autoplaced)
+    (property "Reference" "R47" (at 172.72 92.075 0)
+      (effects (font (size 1.27 1.27)) (justify left))
+    )
+    (property "Value" "2.2k" (at 172.72 94.615 0)
+      (effects (font (size 1.27 1.27)) (justify left))
+    )
+    (property "Footprint" "Resistor_SMD:R_1210_3225Metric_Pad1.30x2.65mm_HandSolder" (at 171.196 92.964 90)
+      (effects (font (size 1.27 1.27)) hide)
+    )
+    (property "Datasheet" "~" (at 170.18 92.71 0)
+      (effects (font (size 1.27 1.27)) hide)
+    )
+    (pin "1")
+    (pin "2")
+    (instances
+      (project "augertapowermanagement"
+        (path "/65134029-dbd2-409a-85a8-13c2a33ff019/8a8c373f-9bc3-4cf7-8f41-4802da916698"
+          (reference "R47") (unit 1)
+        )
+      )

Commit message: update
Parts:
- C14: MANUFACTURER (none) -> B43547A9687M000; Purchase (none) -> https://www.digikey.com/en/products/detail/epcos-tdk-electr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
- JP3, JP4: Purchase NA, JUST pads -> DNP
- R10, R11, R12, R13, R3, R4, R5, R6, R7, R8, R9: MANUFACTURER (none) -> GMR320HJCFAR100
- R47, R48: MANUFACTURER (none) -> RT1210BRD0710KL; Purchase (none) -> https://www.digikey.com/en/products/detail/yageo/RT1210BRD0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
- TP10, TP11, TP12, TP13, TP14, TP4, TP5, TP6, TP7, TP8, TP9: Purchase JUST PAD -> NP
- U10, U11, U12, U13, U3, U4, U5, U6, U7, U8, U9: MANUFACTURER (none) -> INA219AIDR
