File: augertapowermanagement.kicad_pcb (KiCad board)
At the start: 4 copper layers, 316.7 x 183 mm, 82 parts, among them J1 Screw_Terminal_01x02, J10 Screw_Terminal_01x10, J11 Screw_Terminal_01x10, J12 gnd block, J2 76825-0002, J3 USB_A_Stacked, J4 USB_A_Stacked, J5 USB_A_Stacked, J6 USB_A_Stacked, J7 Screw_Terminal_01x08, J8 Screw_Terminal_01x10, J9 5v block, K1 J107F1CS203VDC.80, K2 J107F1CS203VDC.80, SW1 SW_SPDT, U1 LM2596_5v, U10 INA219AxD, U11 INA219AxD, U12 LM2596_5v, U13 LM2596_5v, U14 INA219AxD, U15 INA219AxD, U16 LM2596_11.5v, U17 LM2596_5v, U18 INA219AxD, U19 INA219AxD, U2 ESP32-DEVKITC-32D, U20 LM2596_11.5v, U21 INA219AxD, U22 LM2596_11.5v, U23 INA219AxD, U24 MCP9808_MSOP, U3 INA219AxD, U4 LM2596_5v, U5 LM2596_5v, U6 INA219AxD, U7 INA219AxD, U8 LM2596_5v, U9 LM2596_5v

Commit message: update
Parts:
- JP1, JP2, JP5, JP6: footprint cit:JUMPER_5102TR -> Connector_PinHeader_2.00mm:PinHeader_1x02_P2.00mm_Horizontal
- moved TP5 83.1 mm to (140.2, 184.7)
- moved TP8 62.6 mm to (136.9, 104.5)
- moved U18 47.6 mm to (229.6, 182.2), turned to 180 degrees
- moved JP1 41.8 mm to (124.3, 104.9), turned to 90 degrees
- moved R10 41.1 mm to (228.8, 195.1)
- moved TP17 28.1 mm to (228.8, 153.8)
- moved TP15 27.7 mm to (195.4, 193.2)
- moved TP16 25.1 mm to (264.2, 100.1)
- moved R3 24.5 mm to (276.5, 188.8)
- moved TP12 23.8 mm to (209.3, 101.8)
- moved J5 23.6 mm to (331.2, 56.0)
- moved TP14 23.3 mm to (237.0, 101.8)
- moved U21 22.5 mm to (239.1, 139.6)
- moved J6 21.8 mm to (354.9, 56.0)
- moved C1 21.7 mm to (146.4, 124.1), turned to 90 degrees
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Connections:
- U2 pad 36: Net-(J11-Pad1) -> Net-(J11-Pad3)
- U2 pad 38: Net-(J11-Pad3) -> Net-(J11-Pad1)
Routing:
- net /power_conversion/pi 5v: track 0.00 -> 745.0 mm, vias 0 -> 12
- net /power_conversion/SDA: track 0.00 -> 679.7 mm, vias 0 -> 11
- net /power_conversion/SCL: track 0.00 -> 668.1 mm, vias 0 -> 13
- net Net-(C2-Pad1): track 0.00 -> 213.8 mm
- net /power_conversion/N1: track 0.00 -> 183.7 mm, vias 0 -> 1
- net /power_conversion/N2: track 0.00 -> 182.3 mm, vias 0 -> 1
- net /power_conversion/N3: track 0.00 -> 165.9 mm, vias 0 -> 1
- net /power_conversion/spare2: track 0.00 -> 163.0 mm, vias 0 -> 1
- net -BATT: track 0.00 -> 135.9 mm, vias 0 -> 10
- net /power_conversion/N4: track 0.00 -> 135.3 mm, vias 0 -> 1
- net /power_conversion/pi1: track 0.00 -> 128.5 mm, vias 0 -> 1
- net /power_conversion/battery+: track 0.00 -> 114.8 mm
- net Net-(J8-Pad10): track 0.00 -> 82.5 mm
- net Net-(F1-Pad2): track 0.00 -> 79.0 mm, vias 0 -> 1
- net /power_conversion/spare1: track 0.00 -> 77.7 mm, vias 0 -> 1
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- added copper zone on In1.Cu, net Net-(C2-Pad1)
- added copper zone on F.Cu, net Net-(F1-Pad2)
- added copper zone on In1.Cu, net Net-(F1-Pad2)
Other:
- board size 316.7 x 183 mm -> 315.8 x 183 mm

Commit message: update
Parts:
- moved TP16 3.81 mm to (260.9, 102.1)
- moved J8 3.52 mm to (56.0, 175.5)
- moved JP3 2.61 mm to (208.9, 130.6), turned to 90 degrees
Routing:
- net Net-(R11-Pad2): track 25.3 -> 29.4 mm
- net Net-(J8-Pad8): track 75.2 -> 71.5 mm
- net Net-(J8-Pad5): track 68.1 -> 64.5 mm
- net Net-(J8-Pad7): track 73.2 -> 69.7 mm
- net Net-(J8-Pad6): track 71.9 -> 68.3 mm
- net Net-(J8-Pad3): track 65.3 -> 61.7 mm
- net Net-(J8-Pad1): track 49.8 -> 46.2 mm
- net Net-(J8-Pad4): track 67.1 -> 63.5 mm
- net Net-(J8-Pad2): track 63.5 -> 59.9 mm
- net Net-(J8-Pad10): track 82.5 -> 79.1 mm
- net Net-(J8-Pad9): track 77.1 -> 73.7 mm
- net Net-(JP3-Pad1): track 11.4 -> 8.73 mm

Commit message: update
Changed lines of the file:
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@@
   (net 89 "Net-(R2-Pad2)")
   (net 90 "Net-(K2-Pad1)")
-  (net 91 "Net-(U2-Pad37)")
+  (net 91 "Net-(J11-Pad2)")
   (footprint "Package_SO:SOIC-8_3.9x4.9mm_P1.27mm" (layer "F.Cu")
     (at 355.229026 108.03)
@@
       (net 56 "Net-(J11-Pad3)") (pinfunction "SD1") (pintype "bidirectional"))
     (pad "37" thru_hole circle locked (at 12.7 23.42 90) (size 1.56 1.56) (drill 1.04) (layers *.Cu *.Mask)
-      (net 91 "Net-(U2-Pad37)") (pinfunction "SD0") (pintype "bidirectional"))
+      (net 91 "Net-(J11-Pad2)") (pinfunction "SD0") (pintype "bidirectional"))
     (pad "38" thru_hole circle locked (at 12.7 25.96 90) (size 1.56 1.56) (drill 1.04) (layers *.Cu *.Mask)
       (net 54 "Net-(J11-Pad1)") (pinfunction "CLK") (pintype "input"))
@@
       (net 54 "Net-(J11-Pad1)") (pinfunction "Pin_1") (pintype "passive"))
     (pad "2" thru_hole circle (at 5.08 0 180) (size 2.6 2.6) (drill 1.3) (layers *.Cu *.Mask)
-      (net 91 "Net-(U2-Pad37)") (pinfunction "Pin_2") (pintype "passive"))
+      (net 91 "Net-(J11-Pad2)") (pinfunction "Pin_2") (pintype "passive"))
     (pad "3" thru_hole circle (at 10.16 0 180) (size 2.6 2.6) (drill 1.3) (layers *.Cu *.Mask)
       (net 56 "Net-(J11-Pad3)") (pinfunction "Pin_3") (pintype "passive"))
@@
   (via (at 271.8308 182.3212) (size 1) (drill 0.4) (layers "F.Cu" "B.Cu") (net 2))
   (via (at 238.9632 140.3096) (size 1) (drill 0.4) (layers "F.Cu" "B.Cu") (net 2))
-  (via (at 125.72 191.81) (size 1) (drill 0.4) (layers "F.Cu" "B.Cu") (net 2))
+  (via (at 125.72 191.81) (size 3) (drill 2) (layers "F.Cu" "B.Cu") (net 2))
   (via (at 210.100564 116.543436) (size 1) (drill 0.4) (layers "F.Cu" "B.Cu") (net 2))
   (via (at 350.6724 107.3912) (size 1) (drill 0.4) (layers "F.Cu" "B.Cu") (net 2))
@@
   (segment (start 111.506 76.936) (end 111.506 76.108) (width 0.5) (layer "F.Cu") (net 90))
   (segment (start 128.27 177.8) (end 128.27 160.802974) (width 0.5) (layer "In1.Cu") (net 91))
-  (segment (start 148.780526 211.651) (end 148.780526 198.310526) (width 0.5) (layer "In1.Cu") (net 91))
   (segment (start 148.780526 198.310526) (end 128.27 177.8) (width 0.5) (layer "In1.Cu") (net 91))
   (segment (start 128.27 160.802974) (end 121.003026 153.536) (width 0.5) (layer "In1.Cu") (net 91))
+  (segment (start 148.780526 198.310526) (end 148.780526 211.651) (width 0.5) (layer "In1.Cu") (net 91))
   (zone (net 55) (net_name "Net-(F1-Pad2)") (layer "F.Cu") (hatch edge 0.508)
     (connect_pads (clearance 0.508))

Commit message: update
Connections:
- J7 pad 1: unconnected-(J7-Pad1) -> /power_conversion/routerp
Routing:
- net /power_conversion/routerp: track 53.7 -> 72.3 mm

Commit message: update
Parts:
- JP1, JP2, JP5, JP6: footprint Connector_PinHeader_2.00mm:PinHeader_1x02_P2.00mm_Horizontal -> cit:JUMPER_5102TR
- moved JP5 4.67 mm to (128.8, 67.9), turned to -90 degrees
- moved JP1 3.71 mm to (128.0, 104.5), turned to 0 degrees
- moved JP6 0.88 mm to (155.1, 51.1), turned to 180 degrees
- moved JP2 0.84 mm to (149.3, 69.5), turned to 90 degrees
Routing:
- net Net-(JP1-Pad1): track 52.9 -> 63.0 mm, vias 0 -> 2
- net +BATT: track 0.00 -> 4.79 mm, vias 0 -> 1
- net /power_conversion/battery+: track 114.8 -> 110.4 mm
- net Net-(F1-Pad1): track 12.1 -> 10.3 mm

Commit message: Improved power plane, relay changes, i2c resistor changes
Parts:
- added D1: 1N4007, Diode_THT:D_DO-41_SOD81_P10.16mm_Horizontal, F.Cu at (75.9, 65.4)
- added D2: 1N4007, Diode_THT:D_DO-41_SOD81_P10.16mm_Horizontal, F.Cu at (90.2, 110.7)
- added Q1: 2N3904, Package_TO_SOT_THT:TO-92_HandSolder, F.Cu at (96.4, 125.0)
- K1, K2: footprint cit:Relay_J107F -> Relay_THT:Relay_SPDT_RAYEX-L90S
- R1, R2: value 10k -> 1k; footprint Resistor_SMD:R_1210_3225Metric_Pad1.30x2.65mm_HandSolder -> Resistor_SMD:R_1206_3216Metric_Pad1.30x1.75mm_HandSolder
- R12, R13: value 3.3K -> 5k; footprint Resistor_SMD:R_2512_6332Metric_Pad1.40x3.35mm_HandSolder -> Resistor_SMD:R_1206_3216Metric_Pad1.30x1.75mm_HandSolder
- moved K2 25.2 mm to (95.6, 47.2)
- moved TP1 21.6 mm to (69.3, 72.4), turned to 180 degrees
- moved TP6 10.4 mm to (278.9, 180.1)
- moved R12 3.33 mm to (146.6, 134.2)
- moved K1 1.64 mm to (135.3, 118.2), turned to 180 degrees
- moved F1 1.00 mm to (154.9, 72.3)
Connections:
- net /power_conversion/pi 5v renamed /power_conversion/3v3
- net Net-(F1-Pad2) renamed /power_conversion/Buck in
- K1 pad 14: Net-(K1-Pad14) -> unconnected-(K1-Pad14)
- R1 pad 1: Net-(K1-Pad14) -> -BATT
- R1 pad 2: -BATT -> Net-(U2-Pad21)
- R2 pad 1: -BATT -> Net-(U2-Pad21)
- R2 pad 2: Net-(R2-Pad2) -> Net-(Q1-Pad2)
- SW1 pad 1: Net-(K2-Pad2) -> Net-(K2-PadA2)
- SW1 pad 2: Net-(C2-Pad1) -> +BATT
- SW1 pad 3: Net-(R2-Pad2) -> unconnected-(SW1-Pad3)
- TP4 pad 1: Net-(K1-Pad6) -> Net-(K1-PadA1)
- U2 pad 20: unconnected-(U2-Pad20) -> -BATT
- U2 pad 21: Net-(K1-Pad6) -> Net-(U2-Pad21)
Routing:
- net /power_conversion/Buck in: track 79.0 -> 0.42 mm, vias 1 -> 0
- net Net-(K1-Pad6): track 76.2 -> 0.00 mm
- net /power_conversion/3v3: track 745.3 -> 671.2 mm, vias 12 -> 11
- net Net-(U2-Pad21): track 0.00 -> 46.8 mm
- net Net-(K2-PadA2): track 0.00 -> 38.9 mm
- net /power_conversion/battery+: track 110.4 -> 81.1 mm
- net -BATT: track 135.9 -> 110.5 mm
- net Net-(JP1-Pad1): track 63.0 -> 39.2 mm
- net Net-(K2-Pad2): track 15.4 -> 0.00 mm
- net Net-(K1-Pad14): track 8.84 -> 0.00 mm
- net Net-(K2-Pad1): track 8.46 -> 0.00 mm
- net Net-(K1-PadA1): track 0.00 -> 5.76 mm
- net /power_conversion/SDA: track 679.7 -> 674.3 mm
- net Net-(R2-Pad2): track 5.23 -> 0.00 mm
- net Net-(Q1-Pad2): track 0.00 -> 5.23 mm
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- removed copper zone on In1.Cu, net /power_conversion/Buck in

Commit message: update
Parts:
- moved R2 76.1 mm to (92.4, 123.0)
- moved R1 42.9 mm to (97.8, 126.7), turned to 180 degrees
- moved TP6 11.9 mm to (273.0, 169.8)
- moved TP18 9.27 mm to (347.6, 172.0)
- moved C1 3.91 mm to (150.2, 124.7), turned to -90 degrees
- moved TP17 3.71 mm to (227.0, 150.6)
- moved Q1 3.36 mm to (98.9, 122.7), turned to 90 degrees
Routing:
- net /power_conversion/3v3: track 671.2 -> 753.8 mm, vias 11 -> 13
- net Net-(JP1-Pad1): track 39.2 -> 109.1 mm
- net Net-(K1-PadA1): track 5.76 -> 63.9 mm
- net Net-(C2-Pad1): track 213.8 -> 175.8 mm
- net /power_conversion/battery+: track 81.1 -> 118.1 mm
- net Net-(K2-PadA2): track 38.9 -> 54.3 mm
- net Net-(U2-Pad21): track 46.8 -> 37.7 mm, vias 0 -> 1
- net Net-(R15-Pad2): track 31.2 -> 40.1 mm
- net -BATT: track 110.5 -> 117.3 mm, vias 10 -> 11
- net /power_conversion/SCL: track 668.5 -> 673.0 mm
- net Net-(R14-Pad2): track 59.0 -> 63.0 mm
- net /power_conversion/SDA: track 674.3 -> 676.6 mm

Commit message: updates
Parts:
- removed F1, F2: 1210L900SLPR, Resistor_SMD:R_1210_3225Metric_Pad1.30x2.65mm_HandSolder
- removed JP2, JP6: Jumper_2_Open, cit:JUMPER_5102TR
- removed R16: 10k, Resistor_SMD:R_1210_3225Metric_Pad1.30x2.65mm_HandSolder
- removed TP7, TP8: TestPoint, TestPoint:TestPoint_Plated_Hole_D2.0mm
- added H3: MountingHole, MountingHole:MountingHole_8.4mm_M8, F.Cu at (276.2, 139.3)
- added H4: MountingHole, MountingHole:MountingHole_8.4mm_M8, F.Cu at (324.3, 194.7)
- added H5: MountingHole, MountingHole:MountingHole_8.4mm_M8, F.Cu at (299.9, 51.5)
- added H8: MountingHole, MountingHole:MountingHole_8.4mm_M8, F.Cu at (151.4, 163.4)
- added H9: MountingHole, MountingHole:MountingHole_8.4mm_M8, F.Cu at (60.8, 116.3)
- J1: value Screw_Terminal_01x02 -> Image shown is a representation only. Exact specifications should be obtained from the product data sheet.
- J2: value 76825-0002 -> 0ZCF0200AF2C
Connections:
- JP1 pad 2: /power_conversion/battery+ -> /power_conversion/Buck in
- K1 pad 12: /power_conversion/battery+ -> /power_conversion/Buck in
- U12 pad 1: /power_conversion/Buck in -> unconnected-(U12-Pad1)
Routing:
- net /power_conversion/battery+: track 118.1 -> 0.00 mm
- net /power_conversion/Buck in: track 0.42 -> 110.7 mm
- net Net-(F1-Pad1): track 10.3 -> 0.00 mm
- net -BATT: track 117.3 -> 111.0 mm
- net /power_conversion/SDA: track 676.6 -> 676.0 mm
