File: augertapowermanagement.kicad_pcb (KiCad board)
At the start: 4 copper layers, 315.8 x 183 mm, 83 parts, among them J1 Image shown is a representati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, J10 Screw_Terminal_01x10, J11 Screw_Terminal_01x10, J12 gnd block, J2 0ZCF0200AF2C, J3 USB_A_Stacked, J4 USB_A_Stacked, J5 USB_A_Stacked, J6 USB_A_Stacked, J7 Screw_Terminal_01x08, J8 Screw_Terminal_01x10, J9 5v block, K1 J107F1CS203VDC.80, K2 J107F1CS203VDC.80, Q1 2N3904, SW1 SW_SPDT, U1 LM2596_5v, U10 INA219AxD, U11 INA219AxD, U12 LM2596_5v, U13 LM2596_5v, U14 INA219AxD, U15 INA219AxD, U16 LM2596_11.5v, U17 LM2596_5v, U18 INA219AxD, U19 INA219AxD, U2 ESP32-DEVKITC-32D, U20 LM2596_11.5v, U21 INA219AxD, U22 LM2596_11.5v, U23 INA219AxD, U24 MCP9808_MSOP, U3 INA219AxD, U4 LM2596_5v, U5 LM2596_5v, U6 INA219AxD, U7 INA219AxD, U8 LM2596_5v, U9 LM2596_5v

Commit message: update buck print
Parts:
- H3, H4, H5, H8, H9: footprint MountingHole:MountingHole_8.4mm_M8 -> MountingHole:MountingHole_5mm
- moved TP16 15.9 mm to (276.8, 101.3)
- moved TP10 5.44 mm to (183.6, 103.7)
- moved TP15 4.23 mm to (191.7, 195.2)
- moved TP12 3.69 mm to (213.0, 101.3)
- moved TP14 2.48 mm to (239.4, 101.3)
Routing:
- net Net-(C2-Pad1): track 175.8 -> 191.1 mm
- net Net-(R8-Pad2): track 53.9 -> 41.9 mm
- net Net-(R10-Pad2): track 74.6 -> 63.0 mm
- net -BATT: track 111.0 -> 99.5 mm, vias 11 -> 12
- net Net-(R15-Pad2): track 40.1 -> 46.3 mm
- net Net-(R14-Pad2): track 63.0 -> 57.3 mm
- net Net-(R11-Pad2): track 29.4 -> 23.7 mm
- net Net-(R9-Pad2): track 24.4 -> 29.6 mm
- net Net-(R4-Pad2): track 51.8 -> 47.1 mm
- net Net-(R7-Pad2): track 24.1 -> 26.7 mm
- net Net-(R6-Pad2): track 38.2 -> 36.0 mm
- net Net-(R5-Pad2): track 26.0 -> 24.5 mm

Commit message: hi
Parts:
- removed R12, R13: 5k, Resistor_SMD:R_1206_3216Metric_Pad1.30x1.75mm_HandSolder
- removed TP5: TestPoint, TestPoint:TestPoint_Plated_Hole_D2.0mm
- added D10: 1N5821, Diode_THT:D_DO-201AD_P15.24mm_Horizontal, F.Cu at (1.88, 37.9)
- added D11: 1N5821, Diode_THT:D_DO-201AD_P15.24mm_Horizontal, F.Cu at (1.88, 29.1)
- added D12: 1N5821, Diode_THT:D_DO-201AD_P15.24mm_Horizontal, F.Cu at (1.88, 20.4)
- added D13: 1N5821, Diode_THT:D_DO-201AD_P15.24mm_Horizontal, F.Cu at (23.9, 37.9)
- added D3: 1N5821, Diode_THT:D_DO-201AD_P15.24mm_Horizontal, F.Cu at (23.9, 29.1)
- added D4: 1N5821, Diode_THT:D_DO-201AD_P15.24mm_Horizontal, F.Cu at (23.9, 2.88)
- added D5: 1N5821, Diode_THT:D_DO-201AD_P15.24mm_Horizontal, F.Cu at (23.9, 11.6)
- added D6: 1N5821, Diode_THT:D_DO-201AD_P15.24mm_Horizontal, F.Cu at (1.88, 46.6)
- added D7: 1N5821, Diode_THT:D_DO-201AD_P15.24mm_Horizontal, F.Cu at (23.9, 20.4)
- added D8: 1N5821, Diode_THT:D_DO-201AD_P15.24mm_Horizontal, F.Cu at (1.88, 11.6)
- added D9: 1N5821, Diode_THT:D_DO-201AD_P15.24mm_Horizontal, F.Cu at (1.88, 2.88)
- C1: value 0.1uF -> 680uF
- H3, H4, H5, H8, H9: footprint MountingHole:MountingHole_5mm -> MountingHole:MountingHole_8.4mm_M8
- U1, U12, U13, U17, U4, U5, U8, U9: value LM2596_5v -> LM2596S-ADJ; footprint lm2596:DC_DC_LM2596_small -> Package_TO_SOT_SMD:TO-263-5_TabPin3
- U16, U20, U22: value LM2596_11.5v -> LM2596S-ADJ; footprint lm2596:DC_DC_LM2596_small -> Package_TO_SOT_SMD:TO-263-5_TabPin3
Connections:
- net Net-(C2-Pad1) renamed /Regulator (Adjustable, 3A)10/V_out
- net Net-(JP3-Pad1) renamed /power_conversion/Regulator (Adjustable, 3A)/V_in
- net Net-(JP4-Pad1) renamed /power_conversion/Regulator (Adjustable, 3A)1/V_in
- net Net-(R10-Pad2) renamed /power_conversion/Regulator (Adjustable, 3A)2/V_out
- net Net-(R11-Pad2) renamed /power_conversion/Regulator (Adjustable, 3A)9/V_out
- net Net-(R14-Pad2) renamed /power_conversion/Regulator (Adjustable, 3A)/V_out
- net Net-(R15-Pad2) renamed /power_conversion/Regulator (Adjustable, 3A)1/V_out
- net Net-(R4-Pad2) renamed /power_conversion/Regulator (Adjustable, 3A)5/V_out
- net Net-(R5-Pad2) renamed /power_conversion/Regulator (Adjustable, 3A)6/V_out
- net Net-(R6-Pad2) renamed /power_conversion/Regulator (Adjustable, 3A)4/V_out
- net Net-(R7-Pad2) renamed /power_conversion/Regulator (Adjustable, 3A)7/V_out
- net Net-(R8-Pad2) renamed /power_conversion/Regulator (Adjustable, 3A)3/V_out
- net Net-(R9-Pad2) renamed /power_conversion/Regulator (Adjustable, 3A)8/V_out
- C1 pad 1: /power_conversion/3v3 -> /power_conversion/Buck in
- JP1 pad 1: Net-(JP1-Pad1) -> Net-(JP1-A)
- JP5 pad 2: Net-(JP1-Pad1) -> Net-(JP1-A)
- K1 pad 11: Net-(JP1-Pad1) -> Net-(JP1-A)
- K2 pad 12: unconnected-(K2-Pad12) -> Net-(JP1-A)
- K2 pad 14: Net-(JP1-Pad1) -> unconnected-(K2-Pad14)
- U1 pad 2: -BATT -> Net-(D13-K)
- U12 pad 1: unconnected-(U12-Pad1) -> /power_conversion/Buck in
- U12 pad 2: -BATT -> Net-(D4-K)
- U13 pad 2: -BATT -> Net-(D9-K)
- U16 pad 2: -BATT -> Net-(D3-K)
- U17 pad 2: -BATT -> Net-(D10-K)
- U20 pad 2: -BATT -> Net-(D11-K)
- U22 pad 2: -BATT -> Net-(D12-K)
- U24 pad 1: /power_conversion/SDA -> /power_conversion/3v3
- U24 pad 2: /power_conversion/SCL -> -BATT
- U24 pad 3: unconnected-(U24-Pad3) -> /power_conversion/SCL
- U24 pad 4: -BATT -> /power_conversion/SDA
- U24 pad 8: /power_conversion/3v3 -> unconnected-(U24-A2-Pad8)
- U4 pad 2: -BATT -> Net-(D6-K)
- U5 pad 2: -BATT -> Net-(D7-K)
- U8 pad 2: -BATT -> Net-(D5-K)
- U9 pad 2: -BATT -> Net-(D8-K)
Routing:
- net Net-(JP1-Pad1): track 109.1 -> 0.00 mm, vias 2 -> 0
- net (no net): track 0.00 -> 109.1 mm, vias 0 -> 2

Commit message: finish assigning componets
Parts:
- removed D10, D11, D12, D13, D3, D4, D5, D6, D7, D8, D9: 1N5821, Diode_THT:D_DO-201AD_P15.24mm_Horizontal
- removed H8, H9: MountingHole, MountingHole:MountingHole_8.4mm_M8
- removed JP5: Jumper_2_Open, cit:JUMPER_5102TR
- removed TP15, TP16, TP17, TP18: TestPoint, TestPoint:TestPoint_Plated_Hole_D2.0mm
- added C10: 33u, Capacitor_SMD:C_1206_3216Metric_Pad1.33x1.80mm_HandSolder, F.Cu at (167.3, 204.5)
- added C11: 33u, Capacitor_SMD:C_1206_3216Metric_Pad1.33x1.80mm_HandSolder, F.Cu at (167.3, 207.8)
- added C12: 0.1u X7R, Capacitor_SMD:C_1210_3225Metric_Pad1.33x2.70mm_HandSolder, F.Cu at (209.4, 196.3)
- added C13: 33p, Capacitor_SMD:C_1210_3225Metric_Pad1.33x2.70mm_HandSolder, F.Cu at (209.4, 200.6)
- added C14: 33u, Capacitor_SMD:C_1206_3216Metric_Pad1.33x1.80mm_HandSolder, F.Cu at (195.4, 204.5)
- added C15: 33u, Capacitor_SMD:C_1206_3216Metric_Pad1.33x1.80mm_HandSolder, F.Cu at (195.4, 207.8)
- added C16: 0.1u X7R, Capacitor_SMD:C_1210_3225Metric_Pad1.33x2.70mm_HandSolder, F.Cu at (247.6, 52.6)
- added C17: 33p, Capacitor_SMD:C_1210_3225Metric_Pad1.33x2.70mm_HandSolder, F.Cu at (247.6, 56.8)
- added C18: 33u, Capacitor_SMD:C_1206_3216Metric_Pad1.33x1.80mm_HandSolder, F.Cu at (233.6, 60.7)
- added C19: 33u, Capacitor_SMD:C_1206_3216Metric_Pad1.33x1.80mm_HandSolder, F.Cu at (233.6, 64.1)
- added C20: 0.1u X7R, Capacitor_SMD:C_1210_3225Metric_Pad1.33x2.70mm_HandSolder, F.Cu at (265.5, 168.3)
- added C21: 33p, Capacitor_SMD:C_1210_3225Metric_Pad1.33x2.70mm_HandSolder, F.Cu at (265.5, 172.6)
- added C22: 33u, Capacitor_SMD:C_1206_3216Metric_Pad1.33x1.80mm_HandSolder, F.Cu at (251.5, 176.5)
- added C23: 33u, Capacitor_SMD:C_1206_3216Metric_Pad1.33x1.80mm_HandSolder, F.Cu at (251.5, 179.8)
- added C24: 0.1u X7R, Capacitor_SMD:C_1210_3225Metric_Pad1.33x2.70mm_HandSolder, F.Cu at (209.4, 168.3)
- added C25: 33p, Capacitor_SMD:C_1210_3225Metric_Pad1.33x2.70mm_HandSolder, F.Cu at (209.4, 172.6)
- added C26: 33u, Capacitor_SMD:C_1206_3216Metric_Pad1.33x1.80mm_HandSolder, F.Cu at (195.4, 176.5)
- added C27: 33u, Capacitor_SMD:C_1206_3216Metric_Pad1.33x1.80mm_HandSolder, F.Cu at (195.4, 179.8)
- added C28: 0.1u X7R, Capacitor_SMD:C_1210_3225Metric_Pad1.33x2.70mm_HandSolder, F.Cu at (181.3, 168.3)
- added C29: 33p, Capacitor_SMD:C_1210_3225Metric_Pad1.33x2.70mm_HandSolder, F.Cu at (181.3, 172.6)
- added C3: 680u, Capacitor_THT:CP_Radial_D35.0mm_P10.00mm_SnapIn, F.Cu at (113.1, 174.6)
- added C30: 33u, Capacitor_SMD:C_1206_3216Metric_Pad1.33x1.80mm_HandSolder, F.Cu at (167.3, 176.5)
- added C31: 33u, Capacitor_SMD:C_1206_3216Metric_Pad1.33x1.80mm_HandSolder, F.Cu at (167.3, 179.8)
- added C32: 0.1u X7R, Capacitor_SMD:C_1210_3225Metric_Pad1.33x2.70mm_HandSolder, F.Cu at (265.5, 196.3)
- added C33: 33p, Capacitor_SMD:C_1210_3225Metric_Pad1.33x2.70mm_HandSolder, F.Cu at (265.5, 200.6)
- added C34: 33u, Capacitor_SMD:C_1206_3216Metric_Pad1.33x1.80mm_HandSolder, F.Cu at (251.5, 204.5)
- added C35: 33u, Capacitor_SMD:C_1206_3216Metric_Pad1.33x1.80mm_HandSolder, F.Cu at (251.5, 207.8)
- added C36: 0.1u X7R, Capacitor_SMD:C_1210_3225Metric_Pad1.33x2.70mm_HandSolder, F.Cu at (237.4, 196.3)
- added C37: 33p, Capacitor_SMD:C_1210_3225Metric_Pad1.33x2.70mm_HandSolder, F.Cu at (237.4, 200.6)
- added C38: 33u, Capacitor_SMD:C_1206_3216Metric_Pad1.33x1.80mm_HandSolder, F.Cu at (223.4, 204.5)
- added C39: 33u, Capacitor_SMD:C_1206_3216Metric_Pad1.33x1.80mm_HandSolder, F.Cu at (223.4, 207.8)
- added C4: 0.1u X7R, Capacitor_SMD:C_1210_3225Metric_Pad1.33x2.70mm_HandSolder, F.Cu at (247.6, 80.6)
- added C40: 0.1u X7R, Capacitor_SMD:C_1210_3225Metric_Pad1.33x2.70mm_HandSolder, F.Cu at (237.4, 168.3)
- added C41: 33p, Capacitor_SMD:C_1210_3225Metric_Pad1.33x2.70mm_HandSolder, F.Cu at (237.4, 172.6)
- added C42: 33u, Capacitor_SMD:C_1206_3216Metric_Pad1.33x1.80mm_HandSolder, F.Cu at (223.4, 176.5)
- added C43: 33u, Capacitor_SMD:C_1206_3216Metric_Pad1.33x1.80mm_HandSolder, F.Cu at (223.4, 179.8)
- added C44: 0.1u X7R, Capacitor_SMD:C_1210_3225Metric_Pad1.33x2.70mm_HandSolder, F.Cu at (247.6, 108.6)
- added C45: 33p, Capacitor_SMD:C_1210_3225Metric_Pad1.33x2.70mm_HandSolder, F.Cu at (247.6, 112.8)
- added C46: 33u, Capacitor_SMD:C_1206_3216Metric_Pad1.33x1.80mm_HandSolder, F.Cu at (233.6, 116.7)
- added C47: 33u, Capacitor_SMD:C_1206_3216Metric_Pad1.33x1.80mm_HandSolder, F.Cu at (233.6, 120.1)
- added C5: 33p, Capacitor_SMD:C_1210_3225Metric_Pad1.33x2.70mm_HandSolder, F.Cu at (247.6, 84.8)
- added C6: 33u, Capacitor_SMD:C_1206_3216Metric_Pad1.33x1.80mm_HandSolder, F.Cu at (233.6, 88.7)
- added C7: 33u, Capacitor_SMD:C_1206_3216Metric_Pad1.33x1.80mm_HandSolder, F.Cu at (233.6, 92.1)
- added C8: 0.1u X7R, Capacitor_SMD:C_1210_3225Metric_Pad1.33x2.70mm_HandSolder, F.Cu at (181.3, 196.3)
- added C9: 33p, Capacitor_SMD:C_1210_3225Metric_Pad1.33x2.70mm_HandSolder, F.Cu at (181.3, 200.6)
- added H1: MountingHole, MountingHole:MountingHole_2.5mm, F.Cu at (107.8, 49.8)
- added H2: MountingHole, MountingHole:MountingHole_2.5mm, F.Cu at (107.8, 68.1)
- added JP2: Jumper_2_Open, cit:JUMPER_5102TR, F.Cu at (199.1, 150.1)
- added L1: 5.6u, Inductor_SMD:L_Bourns_SRP1770TA_16.9x16.9mm, F.Cu at (234.5, 77.8)
- added L10: 5.6u, Inductor_SMD:L_Bourns_SRP1770TA_16.9x16.9mm, F.Cu at (224.4, 165.6)
- added L11: 5.6u, Inductor_SMD:L_Bourns_SRP1770TA_16.9x16.9mm, F.Cu at (234.5, 105.8)
- added L2: 5.6u, Inductor_SMD:L_Bourns_SRP1770TA_16.9x16.9mm, F.Cu at (168.3, 193.6)
- added L3: 5.6u, Inductor_SMD:L_Bourns_SRP1770TA_16.9x16.9mm, F.Cu at (196.3, 193.6)
- added L4: 5.6u, Inductor_SMD:L_Bourns_SRP1770TA_16.9x16.9mm, F.Cu at (234.5, 49.8)
- added L5: 5.6u, Inductor_SMD:L_Bourns_SRP1770TA_16.9x16.9mm, F.Cu at (252.4, 165.6)
- added L6: 5.6u, Inductor_SMD:L_Bourns_SRP1770TA_16.9x16.9mm, F.Cu at (196.3, 165.6)
- added L7: 5.6u, Inductor_SMD:L_Bourns_SRP1770TA_16.9x16.9mm, F.Cu at (168.3, 165.6)
- added L8: 5.6u, Inductor_SMD:L_Bourns_SRP1770TA_16.9x16.9mm, F.Cu at (252.4, 193.6)
- added L9: 5.6u, Inductor_SMD:L_Bourns_SRP1770TA_16.9x16.9mm, F.Cu at (224.4, 193.6)
- added R12: 0.1, Resistor_SMD:R_2816_7142Metric_Pad3.20x4.45mm_HandSolder, F.Cu at (151.3, 177.4)
- added R13: 0.1, Resistor_SMD:R_2816_7142Metric_Pad3.20x4.45mm_HandSolder, F.Cu at (151.3, 183.4)
- added R16: 1k, Resistor_SMD:R_1206_3216Metric_Pad1.30x1.75mm_HandSolder, F.Cu at (247.5, 76.8)
- added R17: 18.2k, Resistor_SMD:R_1206_3216Metric_Pad1.30x1.75mm_HandSolder, F.Cu at (181.3, 186.0)
- added R18: 100k, Resistor_SMD:R_1206_3216Metric_Pad1.30x1.75mm_HandSolder, F.Cu at (181.3, 189.3)
- added R19: 1k, Resistor_SMD:R_1206_3216Metric_Pad1.30x1.75mm_HandSolder, F.Cu at (181.3, 192.6)
- added R20: 18.2k, Resistor_SMD:R_1206_3216Metric_Pad1.30x1.75mm_HandSolder, F.Cu at (209.3, 186.0)
- added R21: 100k, Resistor_SMD:R_1206_3216Metric_Pad1.30x1.75mm_HandSolder, F.Cu at (209.3, 189.3)
- added R22: 1k, Resistor_SMD:R_1206_3216Metric_Pad1.30x1.75mm_HandSolder, F.Cu at (209.3, 192.6)
- added R23: 18.2k, Resistor_SMD:R_1206_3216Metric_Pad1.30x1.75mm_HandSolder, F.Cu at (247.5, 42.2)
- added R24: 100k, Resistor_SMD:R_1206_3216Metric_Pad1.30x1.75mm_HandSolder, F.Cu at (247.5, 45.5)
- added R25: 1k, Resistor_SMD:R_1206_3216Metric_Pad1.30x1.75mm_HandSolder, F.Cu at (247.5, 48.8)
- added R26: 18.2k, Resistor_SMD:R_1206_3216Metric_Pad1.30x1.75mm_HandSolder, F.Cu at (265.4, 158.0)
- added R27: 100k, Resistor_SMD:R_1206_3216Metric_Pad1.30x1.75mm_HandSolder, F.Cu at (265.4, 161.3)
- added R28: 1k, Resistor_SMD:R_1206_3216Metric_Pad1.30x1.75mm_HandSolder, F.Cu at (265.4, 164.6)
- added R29: 18.2k, Resistor_SMD:R_1206_3216Metric_Pad1.30x1.75mm_HandSolder, F.Cu at (209.3, 158.0)
- added R30: 100k, Resistor_SMD:R_1206_3216Metric_Pad1.30x1.75mm_HandSolder, F.Cu at (209.3, 161.3)
- added R31: 1k, Resistor_SMD:R_1206_3216Metric_Pad1.30x1.75mm_HandSolder, F.Cu at (209.3, 164.6)
- added R32: 18.2k, Resistor_SMD:R_1206_3216Metric_Pad1.30x1.75mm_HandSolder, F.Cu at (181.3, 158.0)
- added R33: 100k, Resistor_SMD:R_1206_3216Metric_Pad1.30x1.75mm_HandSolder, F.Cu at (181.3, 161.3)
- added R34: 1k, Resistor_SMD:R_1206_3216Metric_Pad1.30x1.75mm_HandSolder, F.Cu at (181.3, 164.6)
- added R35: 18.2k, Resistor_SMD:R_1206_3216Metric_Pad1.30x1.75mm_HandSolder, F.Cu at (265.4, 186.0)
- added R36: 100k, Resistor_SMD:R_1206_3216Metric_Pad1.30x1.75mm_HandSolder, F.Cu at (265.4, 189.3)
- added R37: 1k, Resistor_SMD:R_1206_3216Metric_Pad1.30x1.75mm_HandSolder, F.Cu at (265.4, 192.6)
- added R38: 18.2k, Resistor_SMD:R_1206_3216Metric_Pad1.30x1.75mm_HandSolder, F.Cu at (237.4, 186.0)
- added R39: 100k, Resistor_SMD:R_1206_3216Metric_Pad1.30x1.75mm_HandSolder, F.Cu at (237.4, 189.3)
- added R40: 1k, Resistor_SMD:R_1206_3216Metric_Pad1.30x1.75mm_HandSolder, F.Cu at (237.4, 192.6)
- added R41: 18.2k, Resistor_SMD:R_1206_3216Metric_Pad1.30x1.75mm_HandSolder, F.Cu at (237.4, 158.0)
- added R42: 100k, Resistor_SMD:R_1206_3216Metric_Pad1.30x1.75mm_HandSolder, F.Cu at (237.4, 161.3)
- added R43: 1k, Resistor_SMD:R_1206_3216Metric_Pad1.30x1.75mm_HandSolder, F.Cu at (237.4, 164.6)
- added R44: 18.2k, Resistor_SMD:R_1206_3216Metric_Pad1.30x1.75mm_HandSolder, F.Cu at (247.5, 98.2)
- added R45: 100k, Resistor_SMD:R_1206_3216Metric_Pad1.30x1.75mm_HandSolder, F.Cu at (247.5, 101.5)
- added R46: 1k, Resistor_SMD:R_1206_3216Metric_Pad1.30x1.75mm_HandSolder, F.Cu at (247.5, 104.8)
- added RV1: 50k, Potentiometer_SMD:Potentiometer_Bourns_3314J_Vertical, F.Cu at (227.5, 90.8)
- added RV10: 50k, Potentiometer_SMD:Potentiometer_Bourns_3314J_Vertical, F.Cu at (217.4, 178.6)
- added RV11: 50k, Potentiometer_SMD:Potentiometer_Bourns_3314J_Vertical, F.Cu at (227.5, 118.8)
- added RV2: 50k, Potentiometer_SMD:Potentiometer_Bourns_3314J_Vertical, F.Cu at (161.3, 206.6)
- added RV3: 50k, Potentiometer_SMD:Potentiometer_Bourns_3314J_Vertical, F.Cu at (189.3, 206.6)
- added RV4: 50k, Potentiometer_SMD:Potentiometer_Bourns_3314J_Vertical, F.Cu at (227.5, 62.8)
- added RV5: 50k, Potentiometer_SMD:Potentiometer_Bourns_3314J_Vertical, F.Cu at (245.4, 178.6)
- added RV6: 50k, Potentiometer_SMD:Potentiometer_Bourns_3314J_Vertical, F.Cu at (189.3, 178.6)
- added RV7: 50k, Potentiometer_SMD:Potentiometer_Bourns_3314J_Vertical, F.Cu at (161.3, 178.6)
- added RV8: 50k, Potentiometer_SMD:Potentiometer_Bourns_3314J_Vertical, F.Cu at (245.4, 206.6)
- added RV9: 50k, Potentiometer_SMD:Potentiometer_Bourns_3314J_Vertical, F.Cu at (217.4, 206.6)
- added TP2: TestPoint, TestPoint:TestPoint_Plated_Hole_D2.0mm, F.Cu at (112.5, 139.3)
- added TP5: TestPoint, TestPoint:TestPoint_Plated_Hole_D2.0mm, F.Cu at (126.3, 199.9)
- added TP7: TestPoint, TestPoint:TestPoint_Plated_Hole_D2.0mm, F.Cu at (126.3, 209.2)
- added TP8: TestPoint, TestPoint:TestPoint_Plated_Hole_D2.0mm, F.Cu at (131.0, 195.2)
- added U25: L7812, Package_TO_SOT_THT:TO-220-3_Horizontal_TabDown, F.Cu at (101.9, 152.6)
- C1: value 680uF -> 680u; footprint Capacitor_SMD:C_1210_3225Metric_Pad1.33x2.70mm_HandSolder -> Capacitor_THT:CP_Radial_D35.0mm_P10.00mm_SnapIn
- H3, H4, H5: footprint MountingHole:MountingHole_8.4mm_M8 -> MountingHole:MountingHole_2.5mm
- J1: value Image shown is a representation only. Exact specifications should be obtained from the product data sheet. -> 5v block; footprint TerminalBlock_Phoenix:TerminalBlock_Phoenix_MKDS-1,5-2-5.08_1x02_P5.08mm_Horizontal -> TerminalBlock_Phoenix:TerminalBlock_Phoenix_MKDS-1,5-5-5.08_1x05_P5.08mm_Horizontal
- J10, J11: value Screw_Terminal_01x10 -> USB_A_Stacked; footprint TerminalBlock_Phoenix:TerminalBlock_Phoenix_MKDS-1,5-10-5.08_1x10_P5.08mm_Horizontal -> Connector_USB:USB_A_Wuerth_61400826021_Horizontal_Stacked
- J12: value gnd block -> USB_A_Stacked; footprint TerminalBlock_Phoenix:TerminalBlock_Phoenix_MKDS-1,5-5-5.08_1x05_P5.08mm_Horizontal -> Connector_USB:USB_A_Wuerth_61400826021_Horizontal_Stacked
- J2: value 0ZCF0200AF2C -> Image shown is a representation only. Exact specifications should be obtained from the product data sheet.; footprint Connector_Molex:Molex_Mega-Fit_76825-0002_2x01_P5.70mm_Horizontal -> TerminalBlock_Phoenix:TerminalBlock_Phoenix_MKDS-1,5-2-5.08_1x02_P5.08mm_Horizontal
- J3: value USB_A_Stacked -> gnd block; footprint Connector_USB:USB_A_Wuerth_61400826021_Horizontal_Stacked -> TerminalBlock_Phoenix:TerminalBlock_Phoenix_MKDS-1,5-5-5.08_1x05_P5.08mm_Horizontal
- J4: value USB_A_Stacked -> 0ZCF0200AF2C; footprint Connector_USB:USB_A_Wuerth_61400826021_Horizontal_Stacked -> Connector_Molex:Molex_Mini-Fit_Sr_42819-22XX_1x02_P10.00mm_Vertical_ThermalVias
- J5, J6: value USB_A_Stacked -> Screw_Terminal_01x10; footprint Connector_USB:USB_A_Wuerth_61400826021_Horizontal_Stacked -> TerminalBlock_Phoenix:TerminalBlock_Phoenix_MKDS-1,5-10-5.08_1x10_P5.08mm_Horizontal
- J7: value Screw_Terminal_01x08 -> Screw_Terminal_01x10; footprint TerminalBlock_Phoenix:TerminalBlock_Phoenix_PT-1,5-8-5.0-H_1x08_P5.00mm_Horizontal -> TerminalBlock_Phoenix:TerminalBlock_Phoenix_MKDS-1,5-10-5.08_1x10_P5.08mm_Horizontal
- J8: value Screw_Terminal_01x10 -> Screw_Terminal_01x08; footprint TerminalBlock_Phoenix:TerminalBlock_Phoenix_MKDS-1,5-10-5.08_1x10_P5.08mm_Horizontal -> TerminalBlock_Phoenix:TerminalBlock_Phoenix_PT-1,5-8-5.0-H_1x08_P5.00mm_Horizontal
- J9: value 5v block -> USB_A_Stacked; footprint TerminalBlock_Phoenix:TerminalBlock_Phoenix_MKDS-1,5-5-5.08_1x05_P5.08mm_Horizontal -> Connector_USB:USB_A_Wuerth_61400826021_Horizontal_Stacked
- R14: value 0.1 -> 18.2k; footprint Resistor_SMD:R_2816_7142Metric_Pad3.20x4.45mm_HandSolder -> Resistor_SMD:R_1206_3216Metric_Pad1.30x1.75mm_HandSolder
- R15: value 0.1 -> 100k; footprint Resistor_SMD:R_2816_7142Metric_Pad3.20x4.45mm_HandSolder -> Resistor_SMD:R_1206_3216Metric_Pad1.30x1.75mm_HandSolder
- U1: value LM2596S-ADJ -> ESP32-DEVKITC-32D; footprint Package_TO_SOT_SMD:TO-263-5_TabPin3 -> libary:MODULE_ESP32-DEVKITC-32D
- U12, U13, U4, U5, U8, U9: value LM2596S-ADJ -> INA219AxD; footprint Package_TO_SOT_SMD:TO-263-5_TabPin3 -> Package_SO:SOIC-8_3.9x4.9mm_P1.27mm
- U14, U15, U18, U19, U21, U23: value INA219AxD -> LMR51450; footprint Package_SO:SOIC-8_3.9x4.9mm_P1.27mm -> LMR51:WSON_SDRRR_TEX-M
- U16, U17, U20, U22: value LM2596S-ADJ -> LMR51450; footprint Package_TO_SOT_SMD:TO-263-5_TabPin3 -> LMR51:WSON_SDRRR_TEX-M
- U2: value ESP32-DEVKITC-32D -> MCP9808_MSOP; footprint libary:MODULE_ESP32-DEVKITC-32D -> Connector_PinSocket_2.54mm:PinSocket_1x08_P2.54mm_Vertical
- U24: value MCP9808_MSOP -> LMR51450; footprint Connector_PinSocket_2.54mm:PinSocket_1x08_P2.54mm_Vertical -> LMR51:WSON_SDRRR_TEX-M
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Connections:
- C1 pad 1: /power_conversion/Buck in -> +BATT
- D2 pad 1: +BATT -> +12C
- J1 pad 1: -BATT -> /Regulator (Adjustable, 3A)10/V_out
- J1 pad 2: +BATT -> /Regulator (Adjustable, 3A)10/V_out
- J10 pad 1: Net-(J10-Pin_1) -> /power_conversion/pi2
- J10 pad 2: Net-(J10-Pin_2) -> unconnected-(J10-D1--Pad2)
- J10 pad 3: Net-(J10-Pin_3) -> unconnected-(J10-D1+-Pad3)
- J10 pad 4: Net-(J10-Pin_4) -> -BATT
- J10 pad 5: Net-(J10-Pin_5) -> /power_conversion/pi1
- J10 pad 6: Net-(J10-Pin_6) -> unconnected-(J10-D2--Pad6)
- J10 pad 7: Net-(J10-Pin_7) -> unconnected-(J10-D2+-Pad7)
- J10 pad 8: Net-(J10-Pin_8) -> -BATT
- J10 pad 9: Net-(J10-Pin_9) -> -BATT
- J11 pad 1: Net-(J11-Pin_1) -> /power_conversion/N1
- J11 pad 2: Net-(J11-Pin_2) -> unconnected-(J11-D1--Pad2)
- J11 pad 3: Net-(J11-Pin_3) -> unconnected-(J11-D1+-Pad3)
- J11 pad 4: Net-(J11-Pin_4) -> -BATT
- J11 pad 5: Net-(J11-Pin_5) -> /power_conversion/N2
- J11 pad 6: Net-(J11-Pin_6) -> unconnected-(J11-D2--Pad6)
- J11 pad 7: Net-(J11-Pin_7) -> unconnected-(J11-D2+-Pad7)
- J11 pad 8: Net-(J11-Pin_8) -> -BATT
- J11 pad 9: Net-(J11-Pin_9) -> -BATT
- J12 pad 1: -BATT -> /power_conversion/spare2
- J12 pad 2: -BATT -> unconnected-(J12-D1--Pad2)
- J12 pad 3: -BATT -> unconnected-(J12-D1+-Pad3)
- J12 pad 5: -BATT -> /power_conversion/pi3
- J3 pad 1: /power_conversion/N4 -> -BATT
- J3 pad 2: unconnected-(J3-D1--Pad2) -> -BATT
- J3 pad 3: unconnected-(J3-D1+-Pad3) -> -BATT
- J3 pad 5: /power_conversion/N3 -> -BATT
- J4 pad 1: /power_conversion/N1 -> -BATT
- J4 pad 2: unconnected-(J4-D1--Pad2) -> +BATT
- J5 pad 1: /power_conversion/spare2 -> Net-(J5-Pin_1)
- J5 pad 2: unconnected-(J5-D1--Pad2) -> Net-(J5-Pin_2)
- J5 pad 3: unconnected-(J5-D1+-Pad3) -> Net-(J5-Pin_3)
- J5 pad 4: -BATT -> Net-(J5-Pin_4)
- J5 pad 5: /power_conversion/pi3 -> Net-(J5-Pin_5)
- J5 pad 6: unconnected-(J5-D2--Pad6) -> Net-(J5-Pin_6)
- J5 pad 7: unconnected-(J5-D2+-Pad7) -> Net-(J5-Pin_7)
- J5 pad 8: -BATT -> Net-(J5-Pin_8)
- J5 pad 9: -BATT -> Net-(J5-Pin_9)
- J6 pad 1: /power_conversion/pi2 -> Net-(J6-Pin_1)
- J6 pad 2: unconnected-(J6-D1--Pad2) -> Net-(J6-Pin_2)
- J6 pad 3: unconnected-(J6-D1+-Pad3) -> Net-(J6-Pin_3)
- J6 pad 4: -BATT -> Net-(J6-Pin_4)
- J6 pad 5: /power_conversion/pi1 -> Net-(J6-Pin_5)
- J6 pad 6: unconnected-(J6-D2--Pad6) -> Net-(J6-Pin_6)
- J6 pad 7: unconnected-(J6-D2+-Pad7) -> Net-(J6-Pin_7)
- J6 pad 8: -BATT -> Net-(J6-Pin_8)
- J6 pad 9: -BATT -> Net-(J6-Pin_9)
- J7 pad 1: /power_conversion/routerp -> -BATT
- J7 pad 2: -BATT -> Net-(J7-Pin_2)
- J7 pad 3: /power_conversion/routerp -> Net-(J7-Pin_3)
- J7 pad 4: -BATT -> Net-(J7-Pin_4)
- J7 pad 5: /power_conversion/spare1 -> Net-(J7-Pin_5)
- J7 pad 6: -BATT -> Net-(J7-Pin_6)
- J7 pad 7: /power_conversion/netpw -> Net-(J7-Pin_7)
- J7 pad 8: -BATT -> Net-(J7-Pin_8)
- J8 pad 1: Net-(J8-Pin_1) -> /power_conversion/routerp
- J8 pad 2: Net-(J8-Pin_2) -> -BATT
- J8 pad 3: Net-(J8-Pin_3) -> /power_conversion/routerp
- J8 pad 4: Net-(J8-Pin_4) -> -BATT
- J8 pad 5: Net-(J8-Pin_5) -> /power_conversion/spare1
- J8 pad 6: Net-(J8-Pin_6) -> -BATT
- J8 pad 7: Net-(J8-Pin_7) -> /power_conversion/netpw
- J8 pad 8: Net-(J8-Pin_8) -> -BATT
- J9 pad 1: /Regulator (Adjustable, 3A)10/V_out -> /power_conversion/N4
- J9 pad 2: /Regulator (Adjustable, 3A)10/V_out -> unconnected-(J9-D1--Pad2)
- J9 pad 3: /Regulator (Adjustable, 3A)10/V_out -> unconnected-(J9-D1+-Pad3)
- J9 pad 4: /Regulator (Adjustable, 3A)10/V_out -> -BATT
- J9 pad 5: /Regulator (Adjustable, 3A)10/V_out -> /power_conversion/N3
- JP1 pad 1: Net-(JP1-A) -> +BATT
- JP1 pad 2: /power_conversion/Buck in -> Net-(JP1-B)
- K1 pad 11: Net-(JP1-A) -> +BATT
- K1 pad 12: /power_conversion/Buck in -> Net-(JP1-B)
- K1 pad A1: Net-(D2-A) -> -BATT
- K1 pad A2: +BATT -> Net-(D1-K)
- K2 pad 11: +BATT -> Net-(JP1-B)
- K2 pad 12: Net-(JP1-A) -> /power_conversion/Buck in
- K2 pad A1: -BATT -> Net-(D2-A)
- K2 pad A2: Net-(D1-K) -> +12C
- R1 pad 2: Net-(U2-IO23) -> Net-(U1-IO23)
- R10 pad 1: /power_conversion/netpw -> /power_conversion/N3
- R10 pad 2: /power_conversion/Regulator (Adjustable, 3A)2/V_out -> /power_conversion/Regulator (Adjustable, 3A)8/V_out
- R11 pad 1: /power_conversion/N4 -> /power_conversion/N1
- R11 pad 2: /power_conversion/Regulator (Adjustable, 3A)9/V_out -> /power_conversion/Regulator (Adjustable, 3A)6/V_out
- R14 pad 1: /power_conversion/spare1 -> Net-(U14-RT)
- R14 pad 2: /power_conversion/Regulator (Adjustable, 3A)/V_out -> -BATT
- R15 pad 1: /power_conversion/spare2 -> /power_conversion/Regulator (Adjustable, 3A)2/V_out
- R15 pad 2: /power_conversion/Regulator (Adjustable, 3A)1/V_out -> Net-(U14-FB)
- R2 pad 1: Net-(U2-IO23) -> Net-(U1-IO23)
- R3 pad 1: /power_conversion/routerp -> /power_conversion/spare1
- R3 pad 2: /power_conversion/Buck in -> /power_conversion/Regulator (Adjustable, 3A)/V_out
- R4 pad 1: /power_conversion/pi1 -> /power_conversion/pi3
- R4 pad 2: /power_conversion/Regulator (Adjustable, 3A)5/V_out -> /power_conversion/Regulator (Adjustable, 3A)3/V_out
- R5 pad 1: /power_conversion/N1 -> /power_conversion/pi1
- R5 pad 2: /power_conversion/Regulator (Adjustable, 3A)6/V_out -> /power_conversion/Regulator (Adjustable, 3A)5/V_out
- R7 pad 1: /power_conversion/N2 -> /power_conversion/netpw
- R7 pad 2: /power_conversion/Regulator (Adjustable, 3A)7/V_out -> /power_conversion/Regulator (Adjustable, 3A)2/V_out
- R8 pad 1: /power_conversion/pi3 -> /power_conversion/spare2
- R8 pad 2: /power_conversion/Regulator (Adjustable, 3A)3/V_out -> /power_conversion/Regulator (Adjustable, 3A)1/V_out
- R9 pad 1: /power_conversion/N3 -> /power_conversion/routerp
- R9 pad 2: /power_conversion/Regulator (Adjustable, 3A)8/V_out -> /power_conversion/Buck in
- SW1 pad 2: +BATT -> +12C
- TP10 pad 1: /power_conversion/Regulator (Adjustable, 3A)6/V_out -> /power_conversion/Buck in
- TP11 pad 1: /power_conversion/Regulator (Adjustable, 3A)4/V_out -> /power_conversion/Regulator (Adjustable, 3A)8/V_out
- TP12 pad 1: /power_conversion/Regulator (Adjustable, 3A)7/V_out -> /power_conversion/Regulator (Adjustable, 3A)6/V_out
- TP13 pad 1: /power_conversion/Regulator (Adjustable, 3A)3/V_out -> /power_conversion/Regulator (Adjustable, 3A)7/V_out
- TP14 pad 1: /power_conversion/Regulator (Adjustable, 3A)8/V_out -> /power_conversion/Regulator (Adjustable, 3A)9/V_out
- TP3 pad 1: /Regulator (Adjustable, 3A)10/V_out -> Net-(D2-A)
- TP4 pad 1: Net-(D2-A) -> /power_conversion/Regulator (Adjustable, 3A)1/V_out
- TP6 pad 1: /power_conversion/Buck in -> /power_conversion/Regulator (Adjustable, 3A)3/V_out
- TP9 pad 1: /power_conversion/Regulator (Adjustable, 3A)5/V_out -> /power_conversion/Regulator (Adjustable, 3A)2/V_out
- U1 pad 1: +BATT -> /power_conversion/3v3
- U1 pad 2: Net-(D13-K) -> Net-(J5-Pin_9)
- U1 pad 3: -BATT -> Net-(J5-Pin_8)
- U1 pad 4: /Regulator (Adjustable, 3A)10/V_out -> Net-(J5-Pin_7)
- U1 pad 5: -BATT -> Net-(J5-Pin_6)
- U10 pad 2: -BATT -> /power_conversion/SDA
- U10 pad 7: /power_conversion/pi2 -> /power_conversion/N3
- U10 pad 8: /power_conversion/Regulator (Adjustable, 3A)4/V_out -> /power_conversion/Regulator (Adjustable, 3A)8/V_out
- U11 pad 1: -BATT -> /power_conversion/SCL
- U11 pad 2: /power_conversion/SDA -> /power_conversion/3v3
- U11 pad 7: /power_conversion/N2 -> /power_conversion/N1
- U11 pad 8: /power_conversion/Regulator (Adjustable, 3A)7/V_out -> /power_conversion/Regulator (Adjustable, 3A)6/V_out
- U12 pad 1: /power_conversion/Buck in -> /power_conversion/SDA
- U12 pad 2: Net-(D4-K) -> /power_conversion/SDA
- U12 pad 3: -BATT -> /power_conversion/SDA
- U12 pad 4: /power_conversion/Regulator (Adjustable, 3A)3/V_out -> /power_conversion/SCL
- U12 pad 5: -BATT -> /power_conversion/3v3
- U13 pad 1: /power_conversion/Buck in -> -BATT
- U13 pad 2: Net-(D9-K) -> /power_conversion/SDA
- U13 pad 3: -BATT -> /power_conversion/SDA
- U13 pad 4: /power_conversion/Regulator (Adjustable, 3A)8/V_out -> /power_conversion/SCL
- U13 pad 5: -BATT -> /power_conversion/3v3
- U14 pad 1: /power_conversion/SDA -> Net-(C4-Pad2)
- U14 pad 2: -BATT -> Net-(C4-Pad2)
- U14 pad 3: /power_conversion/SDA -> Net-(C4-Pad2)
- U14 pad 4: /power_conversion/SCL -> Net-(U14-Boot)
- U14 pad 5: /power_conversion/3v3 -> unconnected-(U14-PG-Pad5)
- U14 pad 6: -BATT -> Net-(U14-RT)
- U14 pad 7: /power_conversion/pi3 -> Net-(U14-FB)
- U14 pad 8: /power_conversion/Regulator (Adjustable, 3A)3/V_out -> -BATT
- U15 pad 1: /power_conversion/3v3 -> Net-(C8-Pad2)
- U15 pad 2: /power_conversion/SDA -> Net-(C8-Pad2)
- U15 pad 3: /power_conversion/SDA -> Net-(C8-Pad2)
- U15 pad 4: /power_conversion/SCL -> Net-(U15-Boot)
- U15 pad 5: /power_conversion/3v3 -> unconnected-(U15-PG-Pad5)
- U15 pad 6: -BATT -> Net-(U15-RT)
- U15 pad 7: /power_conversion/N3 -> Net-(U15-FB)
- U15 pad 8: /power_conversion/Regulator (Adjustable, 3A)8/V_out -> -BATT
- U16 pad 1: /power_conversion/Buck in -> Net-(C12-Pad2)
- U16 pad 2: Net-(D3-K) -> Net-(C12-Pad2)
- U16 pad 3: -BATT -> Net-(C12-Pad2)
- U16 pad 4: /power_conversion/Regulator (Adjustable, 3A)2/V_out -> Net-(U16-Boot)
- U16 pad 5: -BATT -> unconnected-(U16-PG-Pad5)
- U17 pad 1: /power_conversion/Buck in -> Net-(C16-Pad2)
- U17 pad 2: Net-(D10-K) -> Net-(C16-Pad2)
- U17 pad 3: -BATT -> Net-(C16-Pad2)
- U17 pad 4: /power_conversion/Regulator (Adjustable, 3A)9/V_out -> Net-(U17-Boot)
- U17 pad 5: -BATT -> unconnected-(U17-PG-Pad5)
- U18 pad 1: /power_conversion/SCL -> Net-(C20-Pad2)
- U18 pad 2: -BATT -> Net-(C20-Pad2)
- U18 pad 3: /power_conversion/SDA -> Net-(C20-Pad2)
- U18 pad 4: /power_conversion/SCL -> Net-(U18-Boot)
- U18 pad 5: /power_conversion/3v3 -> unconnected-(U18-PG-Pad5)
- U18 pad 6: -BATT -> Net-(U18-RT)
- U18 pad 7: /power_conversion/netpw -> Net-(U18-FB)
- U18 pad 8: /power_conversion/Regulator (Adjustable, 3A)2/V_out -> -BATT
- U19 pad 1: /power_conversion/SDA -> Net-(C24-Pad2)
- U19 pad 2: /power_conversion/SDA -> Net-(C24-Pad2)
- U19 pad 3: /power_conversion/SDA -> Net-(C24-Pad2)
- U19 pad 4: /power_conversion/SCL -> Net-(U19-Boot)
- U19 pad 5: /power_conversion/3v3 -> unconnected-(U19-PG-Pad5)
- U19 pad 6: -BATT -> Net-(U19-RT)
- U19 pad 7: /power_conversion/N4 -> Net-(U19-FB)
- U19 pad 8: /power_conversion/Regulator (Adjustable, 3A)9/V_out -> -BATT
- U2 pad 2: Net-(J10-Pin_9) -> -BATT
- U2 pad 3: Net-(J10-Pin_8) -> /power_conversion/SCL
- U2 pad 4: Net-(J10-Pin_7) -> /power_conversion/SDA
- U2 pad 5: Net-(J10-Pin_6) -> unconnected-(U2-Alert-Pad5)
- U2 pad 6: Net-(J10-Pin_5) -> unconnected-(U2-A0-Pad6)
- U2 pad 7: Net-(J10-Pin_4) -> unconnected-(U2-A1-Pad7)
- U2 pad 8: Net-(J10-Pin_3) -> unconnected-(U2-A2-Pad8)
- U20 pad 1: /power_conversion/Regulator (Adjustable, 3A)/V_in -> Net-(C28-Pad2)
- U20 pad 2: Net-(D11-K) -> Net-(C28-Pad2)
- U20 pad 3: -BATT -> Net-(C28-Pad2)
- U20 pad 4: /power_conversion/Regulator (Adjustable, 3A)/V_out -> Net-(U20-Boot)
- U20 pad 5: -BATT -> unconnected-(U20-PG-Pad5)
- U21 pad 1: -BATT -> Net-(C32-Pad2)
- U21 pad 2: /power_conversion/3v3 -> Net-(C32-Pad2)
- U21 pad 3: /power_conversion/SDA -> Net-(C32-Pad2)
- U21 pad 4: /power_conversion/SCL -> Net-(U21-Boot)
- U21 pad 5: /power_conversion/3v3 -> unconnected-(U21-PG-Pad5)
- U21 pad 6: -BATT -> Net-(U21-RT)
- U21 pad 7: /power_conversion/spare1 -> Net-(U21-FB)
- U21 pad 8: /power_conversion/Regulator (Adjustable, 3A)/V_out -> -BATT
- U22 pad 1: /power_conversion/Regulator (Adjustable, 3A)1/V_in -> Net-(C36-Pad2)
- U22 pad 2: Net-(D12-K) -> Net-(C36-Pad2)
- U22 pad 3: -BATT -> Net-(C36-Pad2)
- U22 pad 4: /power_conversion/Regulator (Adjustable, 3A)1/V_out -> Net-(U22-Boot)
- U22 pad 5: -BATT -> unconnected-(U22-PG-Pad5)
- U23 pad 1: /power_conversion/3v3 -> Net-(C40-Pad2)
- U23 pad 2: /power_conversion/3v3 -> Net-(C40-Pad2)
- U23 pad 3: /power_conversion/SDA -> Net-(C40-Pad2)
- U23 pad 4: /power_conversion/SCL -> Net-(U23-Boot)
- U23 pad 5: /power_conversion/3v3 -> unconnected-(U23-PG-Pad5)
- U23 pad 6: -BATT -> Net-(U23-RT)
- U23 pad 7: /power_conversion/spare2 -> Net-(U23-FB)
- U23 pad 8: /power_conversion/Regulator (Adjustable, 3A)1/V_out -> -BATT
- U24 pad 1: /power_conversion/3v3 -> Net-(C44-Pad2)
- U24 pad 2: -BATT -> Net-(C44-Pad2)
- U24 pad 3: /power_conversion/SCL -> Net-(C44-Pad2)
- U24 pad 4: /power_conversion/SDA -> Net-(U24-Boot)
- U24 pad 6: unconnected-(U24-A0-Pad6) -> Net-(U24-RT)
- U24 pad 7: unconnected-(U24-A1-Pad7) -> Net-(U24-FB)
- U24 pad 8: unconnected-(U24-A2-Pad8) -> -BATT
- U3 pad 1: /power_conversion/SDA -> -BATT
- U3 pad 7: /power_conversion/routerp -> /power_conversion/spare1
- U3 pad 8: /power_conversion/Buck in -> /power_conversion/Regulator (Adjustable, 3A)/V_out
- U4 pad 1: /power_conversion/Buck in -> /power_conversion/SDA
- U4 pad 2: Net-(D6-K) -> -BATT
- U4 pad 3: -BATT -> /power_conversion/SDA
- U4 pad 4: /power_conversion/Regulator (Adjustable, 3A)5/V_out -> /power_conversion/SCL
- U4 pad 5: -BATT -> /power_conversion/3v3
- U5 pad 1: /power_conversion/Buck in -> -BATT
- U5 pad 2: Net-(D7-K) -> -BATT
- U5 pad 3: -BATT -> /power_conversion/SDA
- U5 pad 4: /power_conversion/Regulator (Adjustable, 3A)6/V_out -> /power_conversion/SCL
- U5 pad 5: -BATT -> /power_conversion/3v3
- U6 pad 1: -BATT -> /power_conversion/3v3
- U6 pad 7: /power_conversion/pi1 -> /power_conversion/pi2
- U6 pad 8: /power_conversion/Regulator (Adjustable, 3A)5/V_out -> /power_conversion/Regulator (Adjustable, 3A)4/V_out
- U7 pad 2: /power_conversion/3v3 -> -BATT
- U7 pad 7: /power_conversion/N1 -> /power_conversion/netpw
- U7 pad 8: /power_conversion/Regulator (Adjustable, 3A)6/V_out -> /power_conversion/Regulator (Adjustable, 3A)2/V_out
- U8 pad 1: /power_conversion/Buck in -> /power_conversion/3v3
- U8 pad 2: Net-(D5-K) -> /power_conversion/3v3
- U8 pad 3: -BATT -> /power_conversion/SDA
- U8 pad 4: /power_conversion/Regulator (Adjustable, 3A)4/V_out -> /power_conversion/SCL
- U8 pad 5: -BATT -> /power_conversion/3v3
- U9 pad 1: /power_conversion/Buck in -> /power_conversion/SDA
- U9 pad 2: Net-(D8-K) -> /power_conversion/3v3
- U9 pad 3: -BATT -> /power_conversion/SDA
- U9 pad 4: /power_conversion/Regulator (Adjustable, 3A)7/V_out -> /power_conversion/SCL
- U9 pad 5: -BATT -> /power_conversion/3v3
Routing:
- net /power_conversion/3v3: track 753.8 -> 0.00 mm, vias 13 -> 0
- net /power_conversion/SDA: track 676.0 -> 0.00 mm, vias 11 -> 0
- net /power_conversion/SCL: track 673.0 -> 0.00 mm, vias 13 -> 0
- net /Regulator (Adjustable, 3A)10/V_out: track 191.1 -> 0.00 mm
- net /power_conversion/N1: track 183.7 -> 0.00 mm, vias 1 -> 0
- net /power_conversion/N2: track 182.3 -> 0.00 mm, vias 1 -> 0
- net /power_conversion/N3: track 165.9 -> 0.00 mm, vias 1 -> 0
- net /power_conversion/spare2: track 163.0 -> 0.00 mm, vias 1 -> 0
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- removed copper zone on In1.Cu, net +BATT
- removed copper zone on In2.Cu, net -BATT
- removed copper zone on In1.Cu, net /Regulator (Adjustable, 3A)10/V_out
- removed copper zone on F.Cu, net /power_conversion/Buck in
Other:
- board text removed: "Auger@TA Power Managment Board"
- board text removed: "Design by Robin James at CWRU"

Commit message: start pcb
Parts:
- moved C9 337.7 mm to (1.32, -85.2), turned to 90 degrees
- moved C8 332.4 mm to (14.7, -91.3)
- moved R17 332.4 mm to (14.7, -101.7)
- moved R18 332.4 mm to (14.7, -98.4)
- moved R19 326.6 mm to (1.20, -80.0), turned to 90 degrees
- moved U15 326.6 mm to (3.05, -73.2), turned to 180 degrees
- moved RV2 325.8 mm to (-4.62, -73.8), turned to 180 degrees
- moved C11 321.8 mm to (1.18, -67.8), turned to 180 degrees
- moved C10 316.6 mm to (1.18, -65.0), turned to 180 degrees
- moved C15 314.3 mm to (59.6, -75.6)
- moved L3 314.3 mm to (60.5, -89.9)
- moved R22 314.3 mm to (73.5, -90.9)
- moved RV3 314.3 mm to (53.5, -76.9)
- moved U16 314.3 mm to (65.8, -78.0)
- moved C12 314.3 mm to (73.6, -87.1)
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Routing:
- added copper zone on B.Cu, net -BATT

Commit message: board progress
Parts:
- JP3: moved to B.Cu
- moved U6 395.7 mm to (340.0, 168.0)
- moved U5 394.5 mm to (322.0, 189.0)
- moved C28 365.6 mm to (251.3, 207.2)
- moved C29 365.6 mm to (251.3, 211.4)
- moved C30 365.6 mm to (237.3, 215.3)
- moved C31 365.6 mm to (237.3, 218.6)
- moved L7 365.6 mm to (238.3, 204.4)
- moved R32 365.6 mm to (251.3, 196.8)
- moved R33 365.6 mm to (251.3, 200.1)
- moved R34 365.6 mm to (251.3, 203.4)
- moved RV7 365.6 mm to (231.3, 217.4)
- moved U20 365.6 mm to (243.5, 216.3)
- moved C18 364.8 mm to (247.0, 175.9)
- moved C19 364.8 mm to (247.0, 179.2)
- moved L4 364.8 mm to (248.0, 165.0)
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Routing:
- net +12C: track 0.00 -> 236.5 mm
- net /Regulator (Adjustable, 3A)10/V_out: track 0.00 -> 155.7 mm
- net Net-(J7-Pin_2): track 0.00 -> 128.9 mm
- net Net-(J7-Pin_3): track 0.00 -> 126.5 mm
- net Net-(J7-Pin_4): track 0.00 -> 125.5 mm
- net Net-(J7-Pin_5): track 0.00 -> 123.0 mm
- net Net-(J7-Pin_6): track 0.00 -> 120.7 mm
- net Net-(J7-Pin_7): track 0.00 -> 119.7 mm
- net Net-(J7-Pin_8): track 0.00 -> 118.3 mm
- net Net-(D1-K): track 0.00 -> 116.7 mm
- net Net-(J7-Pin_9): track 0.00 -> 116.1 mm
- net Net-(J7-Pin_10): track 0.00 -> 113.8 mm
- net /power_conversion/3v3: track 0.00 -> 106.5 mm
- net Net-(JP1-B): track 0.00 -> 97.8 mm
- net Net-(J5-Pin_9): track 0.00 -> 80.9 mm
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- added copper zone on In2.Cu, net +BATT
- added copper zone on F.Cu, net -BATT
- added copper zone on F.Cu, net /Regulator (Adjustable, 3A)10/V_out
- added copper zone on In2.Cu, net /power_conversion/Buck in

Commit message: progress
Parts:
- moved C20 77.3 mm to (288.5, 131.5), turned to 180 degrees
- moved R26 74.7 mm to (294.8, 127.6), turned to 90 degrees
- moved R27 73.0 mm to (289.9, 116.3), turned to -90 degrees
- moved R28 68.4 mm to (293.7, 116.2), turned to -90 degrees
- moved C21 67.8 mm to (293.3, 120.8), turned to 180 degrees
- moved U18 63.9 mm to (289.9, 126.7), turned to 90 degrees
- moved C22 63.5 mm to (282.1, 116.5), turned to -90 degrees
- moved C43 59.4 mm to (285.0, 87.6), turned to -90 degrees
- moved C23 59.1 mm to (286.2, 116.5), turned to -90 degrees
- moved RV5 57.4 mm to (283.1, 123.0), turned to 90 degrees
- moved JP4 54.7 mm to (286.1, 103.1), turned to -90 degrees
- moved C42 54.4 mm to (289.1, 87.7), turned to -90 degrees
- moved C41 48.7 mm to (297.4, 94.6), turned to -90 degrees
- moved R42 48.3 mm to (293.4, 87.8), turned to -90 degrees
- moved R43 48.0 mm to (297.3, 87.6), turned to -90 degrees
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Routing:
- net /power_conversion/Regulator (Adjustable, 3A)6/V_out: track 0.00 -> 102.4 mm
- net /power_conversion/Regulator (Adjustable, 3A)7/V_out: track 0.00 -> 79.2 mm
- net /power_conversion/Regulator (Adjustable, 3A)1/V_out: track 0.00 -> 57.6 mm
- net /power_conversion/pi3: track 0.00 -> 46.0 mm
- net /power_conversion/N2: track 0.00 -> 36.8 mm
- net Net-(C20-Pad2): track 0.00 -> 29.1 mm
- net /power_conversion/Regulator (Adjustable, 3A)3/V_out: track 24.2 -> 51.3 mm
- net -BATT: track 34.7 -> 60.2 mm, vias 6 -> 14
- net Net-(U15-FB): track 0.00 -> 24.0 mm, vias 0 -> 3
- net Net-(C8-Pad2): track 0.00 -> 20.3 mm
- net Net-(C40-Pad2): track 0.00 -> 18.9 mm
- net Net-(C24-Pad2): track 0.00 -> 17.2 mm
- net /power_conversion/SDA: track 0.00 -> 16.6 mm
- net /power_conversion/spare2: track 0.00 -> 16.1 mm
- net Net-(U18-FB): track 0.00 -> 15.0 mm
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
Commit message: draft done
Parts:
- added H2: MountingHole, MountingHole:MountingHole_2.5mm, F.Cu at (222.4, 124.4)
- moved H4 251.3 mm to (357.8, 208.0)
- moved H3 163.3 mm to (128.2, 182.0)
- moved H5 160.3 mm to (356.4, 77.0)
- moved C15 151.5 mm to (355.6, 120.0), turned to 180 degrees
- moved C14 148.9 mm to (355.6, 123.4), turned to 180 degrees
- moved RV3 146.5 mm to (344.6, 120.0)
- moved L3 133.8 mm to (349.6, 144.8)
- moved R21 129.7 mm to (355.6, 127.4), turned to 180 degrees
- moved R22 129.6 mm to (355.6, 131.2), turned to 180 degrees
- moved U16 128.4 mm to (341.8, 129.6), turned to 180 degrees
- moved C13 127.6 mm to (351.2, 131.4), turned to -90 degrees
- moved C12 121.2 mm to (346.2, 132.6), turned to -90 degrees
- moved R20 121.0 mm to (347.4, 127.2)
- moved U2 114.3 mm to (230.1, 218.6), turned to -90 degrees
- moved H1 99.5 mm to (74.4, 105.0)
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Routing:
- net /power_conversion/3v3: track 119.8 -> 897.8 mm, vias 0 -> 11
- net /power_conversion/SDA: track 16.6 -> 613.5 mm, vias 0 -> 10
- net /power_conversion/SCL: track 8.75 -> 588.3 mm, vias 0 -> 10
- net Net-(U1-IO23): track 0.00 -> 86.3 mm
- net /power_conversion/Regulator (Adjustable, 3A)8/V_out: track 0.00 -> 71.5 mm
- net /power_conversion/Regulator (Adjustable, 3A)5/V_out: track 0.00 -> 66.2 mm
- net /power_conversion/pi2: track 0.00 -> 59.4 mm
- net /power_conversion/Regulator (Adjustable, 3A)4/V_out: track 0.00 -> 57.5 mm
- net -BATT: track 60.2 -> 116.1 mm, vias 14 -> 18
- net /power_conversion/Regulator (Adjustable, 3A)9/V_out: track 0.00 -> 52.7 mm
- net /power_conversion/pi1: track 0.00 -> 40.6 mm
- net /power_conversion/N4: track 0.00 -> 22.5 mm
- net Net-(C12-Pad2): track 0.00 -> 21.1 mm
- net Net-(U16-FB): track 0.00 -> 20.6 mm
- net Net-(C28-Pad2): track 0.00 -> 20.5 mm
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- added copper zone on In1.Cu, net Net-(D2-A)
Other:
- board size 315.8 x 183 mm -> 315.8 x 183.4 mm
- board text added: "Auger@TA Central Power Managment Board Design By CWRU HEA, Robin James"
