File: augertapowermanagement.kicad_pcb (KiCad board)
At the start: 4 copper layers, 315.8 x 183.4 mm, 182 parts, among them J1 5v block, J10 USB_A_Stacked, J11 USB_A_Stacked, J12 USB_A_Stacked, J2 Image shown is a representati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, J3 gnd block, J4 0ZCF0200AF2C, J5 Screw_Terminal_01x10, J6 Screw_Terminal_01x10, J7 Screw_Terminal_01x10, J8 Screw_Terminal_01x08, J9 USB_A_Stacked, K1 J107F1CS203VDC.80, K2 J107F1CS203VDC.80, Q1 2N3904, SW1 SW_SPDT, U1 ESP32-DEVKITC-32D, U10 INA219AxD, U11 INA219AxD, U12 INA219AxD, U13 INA219AxD, U14 LMR51450, U15 LMR51450, U16 LMR51450, U17 LMR51450, U18 LMR51450, U19 LMR51450, U2 MCP9808_MSOP, U20 LMR51450, U21 LMR51450, U22 LMR51450, U23 LMR51450, U24 LMR51450, U25 L7812, U3 INA219AxD, U4 INA219AxD, U5 INA219AxD, U6 INA219AxD, U7 INA219AxD, U8 INA219AxD, U9 INA219AxD

Commit message: fix lot of errors
Parts:
- removed the H2 at (222.4, 124.4)
- added C48: 4.7u X7R, Capacitor_SMD:C_1210_3225Metric_Pad1.33x2.70mm_HandSolder, F.Cu at (197.6, 57.3)
- added C49: 4.7u X7R, Capacitor_SMD:C_1210_3225Metric_Pad1.33x2.70mm_HandSolder, F.Cu at (280.3, 61.0)
- added C50: 4.7u X7R, Capacitor_SMD:C_1210_3225Metric_Pad1.33x2.70mm_HandSolder, F.Cu at (336.7, 132.4)
- added C51: 4.7u X7R, Capacitor_SMD:C_1210_3225Metric_Pad1.33x2.70mm_HandSolder, F.Cu at (317.2, 154.0)
- added C52: 4.7u X7R, Capacitor_SMD:C_1210_3225Metric_Pad1.33x2.70mm_HandSolder, F.Cu at (282.7, 127.7)
- added C53: 4.7u X7R, Capacitor_SMD:C_1210_3225Metric_Pad1.33x2.70mm_HandSolder, F.Cu at (339.5, 99.2)
- added C54: 4.7u X7R, Capacitor_SMD:C_1210_3225Metric_Pad1.33x2.70mm_HandSolder, F.Cu at (252.5, 188.9)
- added C55: 4.7u X7R, Capacitor_SMD:C_1210_3225Metric_Pad1.33x2.70mm_HandSolder, F.Cu at (293.5, 159.9)
- added C56: 4.7u X7R, Capacitor_SMD:C_1210_3225Metric_Pad1.33x2.70mm_HandSolder, F.Cu at (244.6, 89.4)
- added C57: 4.7u X7R, Capacitor_SMD:C_1210_3225Metric_Pad1.33x2.70mm_HandSolder, F.Cu at (284.8, 99.8)
- added C58: 4.7u X7R, Capacitor_SMD:C_1210_3225Metric_Pad1.33x2.70mm_HandSolder, F.Cu at (105.8, 145.4)
- added C59: 10u, Capacitor_SMD:C_1210_3225Metric_Pad1.33x2.70mm_HandSolder, F.Cu at (55.2, 44.5)
- added C60: 4.7u X7R, Capacitor_SMD:C_1210_3225Metric_Pad1.33x2.70mm_HandSolder, F.Cu at (197.7, 60.8)
- added C61: 4.7u X7R, Capacitor_SMD:C_1210_3225Metric_Pad1.33x2.70mm_HandSolder, F.Cu at (285.7, 59.5)
- added C62: 4.7u X7R, Capacitor_SMD:C_1210_3225Metric_Pad1.33x2.70mm_HandSolder, F.Cu at (336.6, 129.0)
- added C63: 4.7u X7R, Capacitor_SMD:C_1210_3225Metric_Pad1.33x2.70mm_HandSolder, F.Cu at (317.1, 157.9)
- added C64: 4.7u X7R, Capacitor_SMD:C_1210_3225Metric_Pad1.33x2.70mm_HandSolder, F.Cu at (282.7, 132.4)
- added C65: 4.7u X7R, Capacitor_SMD:C_1210_3225Metric_Pad1.33x2.70mm_HandSolder, F.Cu at (342.0, 77.5)
- added C66: 4.7u X7R, Capacitor_SMD:C_1210_3225Metric_Pad1.33x2.70mm_HandSolder, F.Cu at (256.5, 189.1)
- added C67: 4.7u X7R, Capacitor_SMD:C_1210_3225Metric_Pad1.33x2.70mm_HandSolder, F.Cu at (293.5, 155.6)
- added C68: 4.7u X7R, Capacitor_SMD:C_1210_3225Metric_Pad1.33x2.70mm_HandSolder, F.Cu at (244.7, 92.9)
- added C69: 4.7u X7R, Capacitor_SMD:C_1210_3225Metric_Pad1.33x2.70mm_HandSolder, F.Cu at (284.6, 95.3)
- added C70: 4.7u X7R, Capacitor_SMD:C_1210_3225Metric_Pad1.33x2.70mm_HandSolder, F.Cu at (109.7, 145.2)
- added H6: MountingHole, MountingHole:MountingHole_2.5mm, F.Cu at (228.1, 150.0)
- added R47: 2.2k, Resistor_SMD:R_1210_3225Metric_Pad1.30x2.65mm_HandSolder, F.Cu at (303.0, 196.1)
- added R48: 2.2k, Resistor_SMD:R_1210_3225Metric_Pad1.30x2.65mm_HandSolder, F.Cu at (272.7, 214.1)
- added R49: 18.2k, Resistor_SMD:R_1206_3216Metric_Pad1.30x1.75mm_HandSolder, F.Cu at (210.4, 68.6)
- added R50: 18.2k, Resistor_SMD:R_1206_3216Metric_Pad1.30x1.75mm_HandSolder, F.Cu at (288.3, 80.5)
- added R51: 18.2k, Resistor_SMD:R_1206_3216Metric_Pad1.30x1.75mm_HandSolder, F.Cu at (350.0, 119.5)
- added R52: 18.2k, Resistor_SMD:R_1206_3216Metric_Pad1.30x1.75mm_HandSolder, F.Cu at (332.2, 137.1)
- added R53: 18.2k, Resistor_SMD:R_1206_3216Metric_Pad1.30x1.75mm_HandSolder, F.Cu at (277.4, 120.2)
- added R54: 18.2k, Resistor_SMD:R_1206_3216Metric_Pad1.30x1.75mm_HandSolder, F.Cu at (346.4, 99.1)
- added R55: 18.2k, Resistor_SMD:R_1206_3216Metric_Pad1.30x1.75mm_HandSolder, F.Cu at (277.1, 196.6)
- added R56: 18.2k, Resistor_SMD:R_1206_3216Metric_Pad1.30x1.75mm_HandSolder, F.Cu at (301.2, 143.8)
- added R57: 18.2k, Resistor_SMD:R_1206_3216Metric_Pad1.30x1.75mm_HandSolder, F.Cu at (228.3, 82.0)
- added R58: 18.2k, Resistor_SMD:R_1206_3216Metric_Pad1.30x1.75mm_HandSolder, F.Cu at (284.4, 91.7)
- added R59: 18.2k, Resistor_SMD:R_1206_3216Metric_Pad1.30x1.75mm_HandSolder, F.Cu at (96.8, 157.5)
- RV1, RV10, RV11, RV2, RV3, RV4, RV5, RV6, RV7, RV8, RV9: value 50k -> 2k
- moved RV7 35.8 mm to (271.1, 193.6), turned to -90 degrees
- moved C31 32.0 mm to (273.4, 203.2), turned to 90 degrees
- moved R32 29.1 mm to (266.4, 193.6), turned to 90 degrees
- moved L9 28.1 mm to (256.4, 81.8)
- moved U20 24.3 mm to (262.1, 193.9), turned to 90 degrees
- moved R33 23.9 mm to (269.4, 203.6), turned to 90 degrees
- moved C29 22.8 mm to (267.0, 198.8), turned to 0 degrees
- moved L7 20.8 mm to (248.7, 204.4), turned to -90 degrees
- moved U25 20.6 mm to (67.7, 63.9), turned to 0 degrees
- moved R34 16.4 mm to (265.6, 203.6), turned to 90 degrees
- moved C28 14.8 mm to (260.9, 198.6), turned to 180 degrees
- moved C36 10.9 mm to (238.9, 81.8)
- moved C38 10.9 mm to (228.5, 75.5)
- moved R40 10.9 mm to (235.2, 75.5)
- moved U22 10.9 mm to (238.7, 87.5)
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Connections:
- RV1 pad 1: -BATT -> Net-(R49-Pad1)
- RV10 pad 1: -BATT -> Net-(R58-Pad1)
- RV11 pad 1: -BATT -> Net-(R59-Pad1)
- RV2 pad 1: -BATT -> Net-(R50-Pad1)
- RV3 pad 1: -BATT -> Net-(R51-Pad1)
- RV4 pad 1: -BATT -> Net-(R52-Pad1)
- RV5 pad 1: -BATT -> Net-(R53-Pad1)
- RV6 pad 1: -BATT -> Net-(R54-Pad1)
- RV7 pad 1: -BATT -> Net-(R55-Pad1)
- RV8 pad 1: -BATT -> Net-(R56-Pad1)
- RV9 pad 1: -BATT -> Net-(R57-Pad1)
Routing:
- net /power_conversion/Buck in: track 40.8 -> 130.6 mm
- net Net-(U14-RT): track 57.5 -> 14.5 mm, vias 0 -> 2
- net +12C: track 236.5 -> 199.3 mm
- net -BATT: track 116.1 -> 145.9 mm, vias 18 -> 86
- net Net-(C36-Pad2): track 51.5 -> 25.5 mm
- net /power_conversion/SDA: track 613.5 -> 631.6 mm, vias 10 -> 11
- net /power_conversion/3v3: track 897.8 -> 910.4 mm, vias 11 -> 12
- net /power_conversion/Regulator (Adjustable, 3A)1/V_in: track 4.50 -> 15.6 mm
- net +BATT: track 20.7 -> 28.3 mm
- net /power_conversion/Regulator (Adjustable, 3A)/V_in: track 4.33 -> 10.4 mm
- net /power_conversion/Regulator (Adjustable, 3A)/V_out: track 42.3 -> 48.0 mm
- net /power_conversion/SCL: track 588.3 -> 593.2 mm
- net Net-(C28-Pad2): track 20.5 -> 16.2 mm
- net Net-(R55-Pad1): track 0.00 -> 4.12 mm
- net Net-(R50-Pad1): track 0.00 -> 3.99 mm
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
Commit message: fixes
Parts:
- added C71: 10u, Capacitor_SMD:C_1210_3225Metric_Pad1.33x2.70mm_HandSolder, F.Cu at (266.4, 52.3)
- added C72: 10u, Capacitor_SMD:C_1210_3225Metric_Pad1.33x2.70mm_HandSolder, F.Cu at (362.2, 60.5)
- added C73: 10u, Capacitor_SMD:C_1210_3225Metric_Pad1.33x2.70mm_HandSolder, F.Cu at (349.5, 170.7)
- added C74: 10u, Capacitor_SMD:C_1210_3225Metric_Pad1.33x2.70mm_HandSolder, F.Cu at (304.8, 200.7)
- R49, R50, R51, R52, R53, R54, R55, R56, R57, R58, R59: value 18.2k -> 10k
- RV1, RV10, RV11, RV2, RV3, RV4, RV5, RV6, RV7, RV8, RV9: value 2k -> 25k
Routing:
- net /power_conversion/3v3: track 910.4 -> 920.9 mm, vias 12 -> 14
- net /Regulator (Adjustable, 3A)10/V_out: track 155.7 -> 164.8 mm
- net /power_conversion/Buck in: track 130.6 -> 133.6 mm, vias 10 -> 37
- net /power_conversion/SCL: track 593.2 -> 593.8 mm
- net -BATT: track 145.9 -> 146.4 mm, vias 86 -> 202

Commit message: update
Changed lines of the file:
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@@
   (paper "A3")
   (layers
-    (0 "F.Cu" signal)
-    (1 "In1.Cu" signal)
-    (2 "In2.Cu" signal)
-    (31 "B.Cu" signal)
+    (0 "F.Cu" power)
+    (1 "In1.Cu" power)
+    (2 "In2.Cu" power)
+    (31 "B.Cu" power)
     (32 "B.Adhes" user "B.Adhesive")
     (33 "F.Adhes" user "F.Adhesive")
@@
     (fp_line (start 1.6 1.25) (end -1.6 1.25)
       (stroke (width 0.1) (type solid)) (layer "F.Fab"))
-    (pad "1" smd roundrect (at -1.5625 0 270) (size 1.325 2.7) (layers "F.Cu" "F.Paste" "F.Mask") (roundrect_rratio 0.188679)
+    (pad "1" smd roundrect (at -1.5625 0 270) (size 1.325 2.7) (layers "F.Cu" "F.Paste" "F.Mask") (roundrect_rratio 0.1886792453)
       (net 1 "/power_conversion/3v3") (pintype "passive"))
-    (pad "2" smd roundrect (at 1.5625 0 270) (size 1.325 2.7) (layers "F.Cu" "F.Paste" "F.Mask") (roundrect_rratio 0.188679)
+    (pad "2" smd roundrect (at 1.5625 0 270) (size 1.325 2.7) (layers "F.Cu" "F.Paste" "F.Mask") (roundrect_rratio 0.1886792453)
       (net 2 "-BATT") (pintype "passive"))
     (model "${KICAD6_3DMODEL_DIR}/Capacitor_SMD.3dshapes/C_1210_3225Metric.wrl"
@@
     (fp_line (start 1.6 1.25) (end -1.6 1.25)
       (stroke (width 0.1) (type solid)) (layer "F.Fab"))
-    (pad "1" smd roundrect (at -1.5625 0) (size 1.325 2.7) (layers "F.Cu" "F.Paste" "F.Mask") (roundrect_rratio 0.188679)
+    (pad "1" smd roundrect (at -1.5625 0) (size 1.325 2.7) (layers "F.Cu" "F.Paste" "F.Mask") (roundrect_rratio 0.1886792453)
       (net 1 "/power_conversion/3v3") (pintype "passive"))
-    (pad "2" smd roundrect (at 1.5625 0) (size 1.325 2.7) (layers "F.Cu" "F.Paste" "F.Mask") (roundrect_rratio 0.188679)
+    (pad "2" smd roundrect (at 1.5625 0) (size 1.325 2.7) (layers "F.Cu" "F.Paste" "F.Mask") (roundrect_rratio 0.1886792453)
       (net 2 "-BATT") (pintype "passive"))
     (model "${KICAD6_3DMODEL_DIR}/Capacitor_SMD.3dshapes/C_1210_3225Metric.wrl"
@@
     (fp_line (start 1.6 1.25) (end -1.6 1.25)
       (stroke (width 0.1) (type solid)) (layer "F.Fab"))
-    (pad "1" smd roundrect (at -1.5625 0) (size 1.325 2.7) (layers "F.Cu" "F.Paste" "F.Mask") (roundrect_rratio 0.188679)
+    (pad "1" smd roundrect (at -1.5625 0) (size 1.325 2.7) (layers "F.Cu" "F.Paste" "F.Mask") (roundrect_rratio 0.1886792453)
       (net 1 "/power_conversion/3v3") (pintype "passive"))
-    (pad "2" smd roundrect (at 1.5625 0) (size 1.325 2.7) (layers "F.Cu" "F.Paste" "F.Mask") (roundrect_rratio 0.188679)
+    (pad "2" smd roundrect (at 1.5625 0) (size 1.325 2.7) (layers "F.Cu" "F.Paste" "F.Mask") (roundrect_rratio 0.1886792453)
       (net 2 "-BATT") (pintype "passive"))
     (model "${KICAD6_3DMODEL_DIR}/Capacitor_SMD.3dshapes/C_1210_3225Metric.wrl"
@@
     (fp_line (start 1.6 1.25) (end -1.6 1.25)
       (stroke (width 0.1) (type solid)) (layer "F.Fab"))
-    (pad "1" smd roundrect (at -1.5625 0 270) (size 1.325 2.7) (layers "F.Cu" "F.Paste" "F.Mask") (roundrect_rratio 0.188679)
+    (pad "1" smd roundrect (at -1.5625 0 270) (size 1.325 2.7) (layers "F.Cu" "F.Paste" "F.Mask") (roundrect_rratio 0.1886792453)
       (net 1 "/power_conversion/3v3") (pintype "passive"))
-    (pad "2" smd roundrect (at 1.5625 0 270) (size 1.325 2.7) (layers "F.Cu" "F.Paste" "F.Mask") (roundrect_rratio 0.188679)
+    (pad "2" smd roundrect (at 1.5625 0 270) (size 1.325 2.7) (layers "F.Cu" "F.Paste" "F.Mask") (roundrect_rratio 0.1886792453)
       (net 2 "-BATT") (pintype "passive"))
     (model "${KICAD6_3DMODEL_DIR}/Capacitor_SMD.3dshapes/C_1210_3225Metric.wrl"

Commit message: update
Parts:
- moved C3 8.98 mm to (176.8, 79.1)
