File: augertapowermanagement.kicad_sch (KiCad schematic)
At the start: 30 parts, among them J1 Screw_Terminal_01x02, J10 Screw_Terminal_01x10, J11 Screw_Terminal_01x10, J12 gnd block, J2 76825-0002, J3 USB_A_Stacked, J4 USB_A_Stacked, J5 USB_A_Stacked, J6 USB_A_Stacked, J7 Screw_Terminal_01x08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

Commit message: update
Parts:
- D1, D2: Purchase (none) -> https://www.digikey.com/en/products/detail/micro-commercial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
- J1: value Screw_Terminal_01x02 -> Image shown is a representation only. Exact specifications should be obtained from the product data sheet.
- J2: value 76825-0002 -> 0ZCF0200AF2C
- K1, K2: Purchase https://www.digikey.com/en/products/detail/cit-relay-and-sw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 -> https://www.digikey.com/en/products/detail/te-connectivity-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
- Q1: Purchase (none) -> https://www.digikey.com/en/products/detail/stmicroelectroni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
- R1, R2: Purchase (none) -> https://www.digikey.com/en/products/detail/stackpole-electr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
Changed lines of the file:
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@@
       (effects (font (size 1.27 1.27)) (justify right))
     )
-    (property "Value" "Screw_Terminal_01x02" (id 1) (at 17.78 15.24 90)
+    (property "Value" "Image shown is a representation only. Exact specifications should be obtained from the product data sheet." (id 1) (at 17.78 15.24 90)
       (effects (font (size 1.27 1.27)) (justify right))
     )
@@
     )
     (property "Datasheet" "~" (id 3) (at 118.11 76.2 0)
+      (effects (font (size 1.27 1.27)) hide)
+    )
+    (property "Purchase" "https://www.digikey.com/en/products/detail/stackpole-electronics-inc/RNCP1206FTD1K00/2240337" (id 4) (at 118.11 76.2 0)
       (effects (font (size 1.27 1.27)) hide)
     )
@@
       (effects (font (size 1.27 1.27)) (justify left) hide)
     )
-    (property "Purchase" "https://www.digikey.com/en/products/detail/cit-relay-and-switch/J107F1CS203VDC-80/14001947" (id 4) (at 64.77 55.88 90)
+    (property "Purchase" "https://www.digikey.com/en/products/detail/te-connectivity-potter-brumfield-relays/T9AS5D12-12/254523" (id 4) (at 64.77 55.88 90)
       (effects (font (size 1.27 1.27)) hide)
     )
@@
       (effects (font (size 1.27 1.27)) (justify left) hide)
     )
-    (property "Purchase" "https://www.digikey.com/en/products/detail/cit-relay-and-switch/J107F1CS203VDC-80/14001947" (id 4) (at 100.33 59.69 90)
+    (property "Purchase" "https://www.digikey.com/en/products/detail/te-connectivity-potter-brumfield-relays/T9AS5D12-12/254523" (id 4) (at 100.33 59.69 90)
       (effects (font (size 1.27 1.27)) hide)
     )
@@
       (effects (font (size 1.27 1.27)) (justify left) hide)
     )
+    (property "Purchase" "https://www.digikey.com/en/products/detail/stmicroelectronics/2N3904/603420" (id 4) (at 121.92 63.5 0)
+      (effects (font (size 1.27 1.27)) hide)
+    )
     (pin "1")
     (pin "2")
@@
       (effects (font (size 1.27 1.27)) hide)
     )
+    (property "Purchase" "https://www.digikey.com/en/products/detail/micro-commercial-co/1N4007GP-TP/2233924" (id 4) (at 63.5 69.85 0)
+      (effects (font (size 1.27 1.27)) hide)
+    )
     (pin "1")
     (pin "2")
@@
       (effects (font (size 1.27 1.27)) hide)
     )
+    (property "Purchase" "https://www.digikey.com/en/products/detail/stackpole-electronics-inc/RNCP1206FTD1K00/2240337" (id 4) (at 121.92 72.39 0)
+      (effects (font (size 1.27 1.27)) hide)
+    )
     (pin "1")
     (pin "2")
@@
     )
     (property "Datasheet" "http://www.vishay.com/docs/88503/1n4001.pdf" (id 3) (at 99.06 74.93 0)
+      (effects (font (size 1.27 1.27)) hide)
+    )
+    (property "Purchase" "https://www.digikey.com/en/products/detail/micro-commercial-co/1N4007GP-TP/2233924" (id 4) (at 99.06 74.93 0)
       (effects (font (size 1.27 1.27)) hide)
     )
@@
       (effects (font (size 1.27 1.27)) (justify right))
     )
-    (property "Value" "76825-0002" (id 1) (at 49.022 23.2922 90)
+    (property "Value" "0ZCF0200AF2C" (id 1) (at 49.022 23.2922 90)
       (effects (font (size 1.27 1.27)) (justify right))
     )
@@
       (reference "D2") (unit 1) (value "1N4007") (footprint "Diode_THT:D_DO-41_SOD81_P10.16mm_Horizontal")
     )
-    (path "/8a8c373f-9bc3-4cf7-8f41-4802da916698/6d8e3d5c-7e48-445f-9603-f7c1bc432955"
-      (reference "F1") (unit 1) (value "1210L900SLPR") (footprint "Resistor_SMD:R_1210_3225Metric_Pad1.30x2.65mm_HandSolder")
-    )
-    (path "/8a8c373f-9bc3-4cf7-8f41-4802da916698/b11dc3f6-cb3f-44f5-898b-d949d476ee5a"
-      (reference "F2") (unit 1) (value "1210L900SLPR") (footprint "Resistor_SMD:R_1210_3225Metric_Pad1.30x2.65mm_HandSolder")
+    (path "/8a8c373f-9bc3-4cf7-8f41-4802da916698/06c6bc2b-d5df-42dd-8701-2d546ead68d8"
+      (reference "F?") (unit 1) (value "Polyfuse") (footprint "")
+    )
+    (path "/8a8c373f-9bc3-4cf7-8f41-4802da916698/0ceeb4d0-735b-4e6b-9f45-88fc1575f7a9"
+      (reference "F?") (unit 1) (value "Polyfuse") (footprint "")
+    )
+    (path "/8a8c373f-9bc3-4cf7-8f41-4802da916698/114425ce-cc70-4848-a6fa-b1b1151a3ec6"
+      (reference "F?") (unit 1) (value "Polyfuse") (footprint "")
+    )
+    (path "/8a8c373f-9bc3-4cf7-8f41-4802da916698/2fef1f59-5fe8-4958-a064-d34c69a58139"
+      (reference "F?") (unit 1) (value "Polyfuse") (footprint "")
+    )
+    (path "/8a8c373f-9bc3-4cf7-8f41-4802da916698/780004b0-9533-4778-b94a-7329e9dda853"
+      (reference "F?") (unit 1) (value "Polyfuse") (footprint "")
+    )
+    (path "/8a8c373f-9bc3-4cf7-8f41-4802da916698/83883f3d-3467-44be-94af-0c6feb053815"
+      (reference "F?") (unit 1) (value "Polyfuse") (footprint "")
+    )
+    (path "/8a8c373f-9bc3-4cf7-8f41-4802da916698/93e08622-ffd3-49f5-ae38-3f2ed2f17625"
+      (reference "F?") (unit 1) (value "Polyfuse") (footprint "")
+    )
+    (path "/8a8c373f-9bc3-4cf7-8f41-4802da916698/a29639d9-23d8-457c-871d-d557a00cbeab"
+      (reference "F?") (unit 1) (value "Polyfuse") (footprint "")
+    )
+    (path "/8a8c373f-9bc3-4cf7-8f41-4802da916698/abded411-de5a-469b-b016-ba4865f0ec15"
+      (reference "F?") (unit 1) (value "Polyfuse") (footprint "")
+    )
+    (path "/8a8c373f-9bc3-4cf7-8f41-4802da916698/cbf52bda-49b7-494e-87f1-cd2f177cb925"
+      (reference "F?") (unit 1) (value "Polyfuse") (footprint "")
+    )
+    (path "/8a8c373f-9bc3-4cf7-8f41-4802da916698/f7978fbc-bc18-40b8-b324-0e42fdcb6360"
+      (reference "F?") (unit 1) (value "Polyfuse") (footprint "")
     )
     (path "/0565831f-1b30-4646-8f44-1aeedcbf4a29"
-      (reference "J1") (unit 1) (value "Screw_Terminal_01x02") (footprint "TerminalBlock_Phoenix:TerminalBlock_Phoenix_MKDS-1,5-2-5.08_1x02_P5.08mm_Horizontal")
+      (reference "J1") (unit 1) (value "Image shown is a representation only. Exact specifications should be obtained from the product data sheet.") (footprint "TerminalBlock_Phoenix:TerminalBlock_Phoenix_MKDS-1,5-2-5.08_1x02_P5.08mm_Horizontal")
     )
     (path "/9fd0cb17-b4d5-4f80-aeda-8a9978760fa2"
-      (reference "J2") (unit 1) (value "76825-0002") (footprint "Connector_Molex:Molex_Mega-Fit_76825-0002_2x01_P5.70mm_Horizontal")
+      (reference "J2") (unit 1) (value "0ZCF0200AF2C") (footprint "Connector_Molex:Molex_Mega-Fit_76825-0002_2x01_P5.70mm_Horizontal")
     )
     (path "/14edb43d-845c-4c8d-9d4b-9b7872f32230"
@@
       (reference "JP1") (unit 1) (value "Jumper_2_Open") (footprint "cit:JUMPER_5102TR")
     )
-    (path "/8a8c373f-9bc3-4cf7-8f41-4802da916698/50a4d4a6-86ed-460b-979f-ababc72cae1c"
-      (reference "JP2") (unit 1) (value "Jumper_2_Open") (footprint "cit:JUMPER_5102TR")
-    )
     (path "/8a8c373f-9bc3-4cf7-8f41-4802da916698/5768f29d-5de4-4595-abf0-f6083c155be3"
       (reference "JP3") (unit 1) (value "Jumper_2_Open") (footprint "Connector_PinHeader_2.00mm:PinHeader_1x02_P2.00mm_Horizontal")
@@
       (reference "JP5") (unit 1) (value "Jumper_2_Open") (footprint "cit:JUMPER_5102TR")
     )
-    (path "/8a8c373f-9bc3-4cf7-8f41-4802da916698/1ed5a3a3-3988-44f5-970d-7e971f9abf8f"
-      (reference "JP6") (unit 1) (value "Jumper_2_Open") (footprint "cit:JUMPER_5102TR")
-    )
     (path "/1347a48f-a9f7-470c-893f-af03f52f8d81"
       (reference "K1") (unit 1) (value "J107F1CS203VDC.80") (footprint "Relay_THT:Relay_SPDT_RAYEX-L90S")
@@
       (reference "TP6") (unit 1) (value "TestPoint") (footprint "TestPoint:TestPoint_Plated_Hole_D2.0mm")
     )
-    (path "/8a8c373f-9bc3-4cf7-8f41-4802da916698/16aa1ab8-e213-456b-95a7-db0db8a30701"
-      (reference "TP7") (unit 1) (value "TestPoint") (footprint "TestPoint:TestPoint_Plated_Hole_D2.0mm")
-    )
-    (path "/8a8c373f-9bc3-4cf7-8f41-4802da916698/7a529dee-c005-4452-892e-c7d1683c627a"
-      (reference "TP8") (unit 1) (value "TestPoint") (footprint "TestPoint:TestPoint_Plated_Hole_D2.0mm")
-    )
     (path "/8a8c373f-9bc3-4cf7-8f41-4802da916698/7f9d0bf1-f44a-42de-888c-c039245505e9"

Commit message: updates
Parts:
- added H3, H4, H5, H8, H9: MountingHole, MountingHole:MountingHole_8.4mm_M8, symbol Mechanical:MountingHole
Changed lines of the file:
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@@
     (pin "1")
+  )
+  (symbol (lib_id "Mechanical:MountingHole") (at 142.24 168.91 0) (unit 1)
+    (in_bom yes) (on_board yes) (fields_autoplaced)
+    (property "Reference" "H8" (id 0) (at 144.78 167.6399 0)
+      (effects (font (size 1.27 1.27)) (justify left))
+    )
+    (property "Value" "MountingHole" (id 1) (at 144.78 170.1799 0)
+      (effects (font (size 1.27 1.27)) (justify left))
+    )
+    (property "Footprint" "MountingHole:MountingHole_8.4mm_M8" (id 2) (at 142.24 168.91 0)
+      (effects (font (size 1.27 1.27)) hide)
+    )
+    (property "Datasheet" "~" (id 3) (at 142.24 168.91 0)
+      (effects (font (size 1.27 1.27)) hide)
+    )
   )
   (symbol (lib_id "power:+BATT") (at 27.94 27.94 270) (unit 1)
@@
     (pin "1")
     (pin "2")
+  )
+  (symbol (lib_id "Mechanical:MountingHole") (at 111.76 176.53 0) (unit 1)
+    (in_bom yes) (on_board yes) (fields_autoplaced)
+    (property "Reference" "H9" (id 0) (at 114.3 175.2599 0)
+      (effects (font (size 1.27 1.27)) (justify left))
+    )
+    (property "Value" "MountingHole" (id 1) (at 114.3 177.7999 0)
+      (effects (font (size 1.27 1.27)) (justify left))
+    )
+    (property "Footprint" "MountingHole:MountingHole_8.4mm_M8" (id 2) (at 111.76 176.53 0)
+      (effects (font (size 1.27 1.27)) hide)
+    )
+    (property "Datasheet" "~" (id 3) (at 111.76 176.53 0)
+      (effects (font (size 1.27 1.27)) hide)
+    )
+  )
+  (symbol (lib_id "Mechanical:MountingHole") (at 130.81 153.67 0) (unit 1)
+    (in_bom yes) (on_board yes) (fields_autoplaced)
+    (property "Reference" "H3" (id 0) (at 133.35 152.3999 0)
+      (effects (font (size 1.27 1.27)) (justify left))
+    )
+    (property "Value" "MountingHole" (id 1) (at 133.35 154.9399 0)
+      (effects (font (size 1.27 1.27)) (justify left))
+    )
+    (property "Footprint" "MountingHole:MountingHole_8.4mm_M8" (id 2) (at 130.81 153.67 0)
+      (effects (font (size 1.27 1.27)) hide)
+    )
+    (property "Datasheet" "~" (id 3) (at 130.81 153.67 0)
+      (effects (font (size 1.27 1.27)) hide)
+    )
   )
   (symbol (lib_id "Diode:1N4007") (at 99.06 74.93 0) (unit 1)
@@
     (pin "9")
   )
+  (symbol (lib_id "Mechanical:MountingHole") (at 154.94 160.02 0) (unit 1)
+    (in_bom yes) (on_board yes) (fields_autoplaced)
+    (property "Reference" "H5" (id 0) (at 157.48 158.7499 0)
+      (effects (font (size 1.27 1.27)) (justify left))
+    )
+    (property "Value" "MountingHole" (id 1) (at 157.48 161.2899 0)
+      (effects (font (size 1.27 1.27)) (justify left))
+    )
+    (property "Footprint" "MountingHole:MountingHole_8.4mm_M8" (id 2) (at 154.94 160.02 0)
+      (effects (font (size 1.27 1.27)) hide)
+    )
+    (property "Datasheet" "~" (id 3) (at 154.94 160.02 0)
+      (effects (font (size 1.27 1.27)) hide)
+    )
+  )
+  (symbol (lib_id "Mechanical:MountingHole") (at 118.11 158.75 0) (unit 1)
+    (in_bom yes) (on_board yes) (fields_autoplaced)
+    (property "Reference" "H4" (id 0) (at 120.65 157.4799 0)
+      (effects (font (size 1.27 1.27)) (justify left))
+    )
+    (property "Value" "MountingHole" (id 1) (at 120.65 160.0199 0)
+      (effects (font (size 1.27 1.27)) (justify left))
+    )
+    (property "Footprint" "MountingHole:MountingHole_8.4mm_M8" (id 2) (at 118.11 158.75 0)
+      (effects (font (size 1.27 1.27)) hide)
+    )
+    (property "Datasheet" "~" (id 3) (at 118.11 158.75 0)
+      (effects (font (size 1.27 1.27)) hide)
+    )
+  )
   (symbol (lib_id "Connector:TestPoint") (at 50.8 78.74 0) (unit 1)
     (in_bom yes) (on_board yes) (fields_autoplaced)
@@
       (reference "D2") (unit 1) (value "1N4007") (footprint "Diode_THT:D_DO-41_SOD81_P10.16mm_Horizontal")
     )
-    (path "/8a8c373f-9bc3-4cf7-8f41-4802da916698/06c6bc2b-d5df-42dd-8701-2d546ead68d8"
-      (reference "F?") (unit 1) (value "Polyfuse") (footprint "")
-    )
-    (path "/8a8c373f-9bc3-4cf7-8f41-4802da916698/0ceeb4d0-735b-4e6b-9f45-88fc1575f7a9"
-      (reference "F?") (unit 1) (value "Polyfuse") (footprint "")
-    )
-    (path "/8a8c373f-9bc3-4cf7-8f41-4802da916698/114425ce-cc70-4848-a6fa-b1b1151a3ec6"
-      (reference "F?") (unit 1) (value "Polyfuse") (footprint "")
-    )
-    (path "/8a8c373f-9bc3-4cf7-8f41-4802da916698/2fef1f59-5fe8-4958-a064-d34c69a58139"
-      (reference "F?") (unit 1) (value "Polyfuse") (footprint "")
-    )
-    (path "/8a8c373f-9bc3-4cf7-8f41-4802da916698/780004b0-9533-4778-b94a-7329e9dda853"
-      (reference "F?") (unit 1) (value "Polyfuse") (footprint "")
-    )
-    (path "/8a8c373f-9bc3-4cf7-8f41-4802da916698/83883f3d-3467-44be-94af-0c6feb053815"
-      (reference "F?") (unit 1) (value "Polyfuse") (footprint "")
-    )
-    (path "/8a8c373f-9bc3-4cf7-8f41-4802da916698/93e08622-ffd3-49f5-ae38-3f2ed2f17625"
-      (reference "F?") (unit 1) (value "Polyfuse") (footprint "")
-    )
-    (path "/8a8c373f-9bc3-4cf7-8f41-4802da916698/a29639d9-23d8-457c-871d-d557a00cbeab"
-      (reference "F?") (unit 1) (value "Polyfuse") (footprint "")
-    )
-    (path "/8a8c373f-9bc3-4cf7-8f41-4802da916698/abded411-de5a-469b-b016-ba4865f0ec15"
-      (reference "F?") (unit 1) (value "Polyfuse") (footprint "")
-    )
-    (path "/8a8c373f-9bc3-4cf7-8f41-4802da916698/cbf52bda-49b7-494e-87f1-cd2f177cb925"
-      (reference "F?") (unit 1) (value "Polyfuse") (footprint "")
-    )
-    (path "/8a8c373f-9bc3-4cf7-8f41-4802da916698/f7978fbc-bc18-40b8-b324-0e42fdcb6360"
-      (reference "F?") (unit 1) (value "Polyfuse") (footprint "")
+    (path "/7a063af9-8404-4ba6-8517-b35030913585"
+      (reference "H3") (unit 1) (value "MountingHole") (footprint "MountingHole:MountingHole_8.4mm_M8")
+    )
+    (path "/a83a8a47-2521-4237-98bd-73a2715c88c6"
+      (reference "H4") (unit 1) (value "MountingHole") (footprint "MountingHole:MountingHole_8.4mm_M8")
+    )
+    (path "/a217261a-11d0-4a81-8ec6-f8dd14eab940"
+      (reference "H5") (unit 1) (value "MountingHole") (footprint "MountingHole:MountingHole_8.4mm_M8")
+    )
+    (path "/677524e1-c21d-4b72-a2e6-34dbe4532d27"
+      (reference "H8") (unit 1) (value "MountingHole") (footprint "MountingHole:MountingHole_8.4mm_M8")
+    )
+    (path "/78cd53a2-2937-4674-bb3d-3388761783a5"
+      (reference "H9") (unit 1) (value "MountingHole") (footprint "MountingHole:MountingHole_8.4mm_M8")
     )
     (path "/0565831f-1b30-4646-8f44-1aeedcbf4a29"

Commit message: 04/13/2023
Connections:
- net at K2.12: now also JP1.1 (A), JP5.2 (B), K1.11
- now unconnected: K2.14
Other:
- note removed: "should I use 2 i2c buses"
