File: augertapowermanagement.kicad_sch (KiCad schematic)
At the start: 35 parts, among them J1 Image shown is a representati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, J10 Screw_Terminal_01x10, J11 Screw_Terminal_01x10, J12 gnd block, J2 0ZCF0200AF2C, J3 USB_A_Stacked, J4 USB_A_Stacked, J5 USB_A_Stacked, J6 USB_A_Stacked, J7 Screw_Terminal_01x08, J8 Screw_Terminal_01x10, J9 5v block, K1 J107F1CS203VDC.80, K2 J107F1CS203VDC.80, Q1 2N3904, SW1 SW_SPDT, U1 LM2596_5v, U2 ESP32-DEVKITC-32D, U24 MCP9808_MSOP

Commit message: hi
Parts:
- removed TP5: TestPoint, TestPoint:TestPoint_Plated_Hole_D2.0mm, symbol Connector:TestPoint
- removed U1: LM2596_5v, lm2596:DC_DC_LM2596_small, symbol powermanagement:YAAJ_DCDC_StepDown_LM2596
- J2: footprint Connector_Molex:Molex_Mega-Fit_76825-0002_2x01_P5.70mm_Horizontal -> Connector_Molex:Molex_Mini-Fit_Sr_42819-22XX_1x02_P10.00mm_Vertical_ThermalVias
Connections:
- net -BATT: now also J8.1 (Pin_1), U2.26 (GND2), U24.2 (GND); no longer U24.4 (GND)
- net power_conversion/3v3: now also U24.1 (VDD); no longer U24.8 (VDD)
- net power_conversion/SCL: now also U24.3 (SCL); no longer U24.2 (SCL)
- net power_conversion/SDA: now also U24.4 (SDA); no longer U24.1 (SDA)
- net Regulator (Adjustable, 3A)10/V_out: now reaches C2.1, J9.1 (Pin_1), J9.2 (Pin_2), J9.3 (Pin_3), J9.4 (Pin_4), J9.5 (Pin_5), TP3.1, U2.19 (EXT_5V)
Other:
- added sheet Regulator (Adjustable, 3A)10 (Adjustable Regulator.kicad_sch)
- note removed: "This is 3.3v not 5v"

Commit message: finish assigning componets
Parts:
- added C1: 680u, Capacitor_THT:CP_Radial_D35.0mm_P10.00mm_SnapIn, symbol Device:C
- added U25: L7812, Package_TO_SOT_THT:TO-220-3_Horizontal_TabDown, symbol Regulator_Linear:L7812
- H1: renamed from H9; footprint MountingHole:MountingHole_8.4mm_M8 -> MountingHole:MountingHole_2.5mm
- H2: renamed from H4; footprint MountingHole:MountingHole_8.4mm_M8 -> MountingHole:MountingHole_2.5mm
- H3, H5: footprint MountingHole:MountingHole_8.4mm_M8 -> MountingHole:MountingHole_2.5mm
- H4: renamed from H8; footprint MountingHole:MountingHole_8.4mm_M8 -> MountingHole:MountingHole_2.5mm
- renumbered J9 to J1, J6 to J10, J4 to J11, J5 to J12, J1 to J2, J12 to J3, J2 to J4, J10 to J5, J11 to J6, J8 to J7, J7 to J8, J3 to J9, JP5 to JP1, JP1 to JP2, K2 to K1, K1 to K2, TP3 to TP2, TP4 to TP3, U2 to U1, U24 to U2
Connections:
- net +BATT: now also C1.1, U25.1 (IN); no longer D2.1 (K), K2.A2, SW1.2 (B)
- net -BATT: now also C1.2, U25.2 (GND)
- new net +12C: D2.1 (K), K2.A2, SW1.2 (B), U25.3 (OUT)

Commit message: fix lot of errors
Parts:
- added C59: 10u, Capacitor_SMD:C_1210_3225Metric_Pad1.33x2.70mm_HandSolder, symbol Device:C
- added H6: MountingHole, MountingHole:MountingHole_2.5mm, symbol Mechanical:MountingHole
Connections:
- net +12C: now also C59.1
- net -BATT: now also C59.2
Changed lines of the file:
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@@
   (junction (at 251.46 50.8) (diameter 0) (color 0 0 0 0)
   )
+  (junction (at 138.43 29.21) (diameter 0) (color 0 0 0 0)
+  )
   (junction (at 196.85 60.96) (diameter 0) (color 0 0 0 0)
   )
@@
   )
   (junction (at 187.96 15.24) (diameter 0) (color 0 0 0 0)
+  )
+  (junction (at 147.32 21.59) (diameter 0) (color 0 0 0 0)
   )
   (junction (at 29.21 162.56) (diameter 0) (color 0 0 0 0)
@@
     (stroke (width 0) (type default))
   )
+  (wire (pts (xy 138.43 29.21) (xy 147.32 29.21))
+    (stroke (width 0) (type default))
+  )
   (wire (pts (xy 127 64.77) (xy 127 95.25))
     (stroke (width 0) (type default))
@@
     (stroke (width 0) (type default))
   )
+  (wire (pts (xy 147.32 21.59) (xy 149.86 21.59))
+    (stroke (width 0) (type default))
+  )
   (wire (pts (xy 172.72 50.8) (xy 172.72 15.24))
     (stroke (width 0) (type default))
@@
     (stroke (width 0) (type default))
   )
-  (wire (pts (xy 146.05 21.59) (xy 149.86 21.59))
+  (wire (pts (xy 146.05 21.59) (xy 147.32 21.59))
     (stroke (width 0) (type default))
   )
@@
         (path "/65134029-dbd2-409a-85a8-13c2a33ff019"
           (reference "J2") (unit 1)
+        )
+      )
+    )
+  )
+  (symbol (lib_id "Device:C") (at 147.32 25.4 0) (unit 1)
+    (in_bom yes) (on_board yes) (dnp no) (fields_autoplaced)
+    (property "Reference" "C59" (at 151.13 24.765 0)
+      (effects (font (size 1.27 1.27)) (justify left))
+    )
+    (property "Value" "10u" (at 151.13 27.305 0)
+      (effects (font (size 1.27 1.27)) (justify left))
+    )
+    (property "Footprint" "Capacitor_SMD:C_1210_3225Metric_Pad1.33x2.70mm_HandSolder" (at 148.2852 29.21 0)
+      (effects (font (size 1.27 1.27)) hide)
+    )
+    (property "Datasheet" "~" (at 147.32 25.4 0)
+      (effects (font (size 1.27 1.27)) hide)
+    )
+    (pin "1")
+    (pin "2")
+    (instances
+      (project "augertapowermanagement"
+        (path "/65134029-dbd2-409a-85a8-13c2a33ff019"
+          (reference "C59") (unit 1)
         )
       )
@@
         )
       )
+    )
+  )
+  (symbol (lib_id "Mechanical:MountingHole") (at 137.16 181.61 0) (unit 1)
+    (in_bom yes) (on_board yes) (dnp no) (fields_autoplaced)
+    (property "Reference" "H6" (at 139.7 180.3399 0)
+      (effects (font (size 1.27 1.27)) (justify left))
+    )
+    (property "Value" "MountingHole" (at 139.7 182.8799 0)
+      (effects (font (size 1.27 1.27)) (justify left))
+    )
+    (property "Footprint" "MountingHole:MountingHole_2.5mm" (at 137.16 181.61 0)
+      (effects (font (size 1.27 1.27)) hide)
+    )
+    (property "Datasheet" "~" (at 137.16 181.61 0)
+      (effects (font (size 1.27 1.27)) hide)
+    )
+    (instances
+      (project "augertapowermanagement"
+        (path "/65134029-dbd2-409a-85a8-13c2a33ff019"
+          (reference "H6") (unit 1)
+        )
+      )

Commit message: fixes
Parts:
- added C71, C72, C73, C74: 10u, Capacitor_SMD:C_1210_3225Metric_Pad1.33x2.70mm_HandSolder, symbol Device:C
Connections:
- net -BATT: now also C71.2, C72.2, C73.2, C74.2
- net power_conversion/3v3: now also C71.1, C72.1, C73.1, C74.1
Changed lines of the file:
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@@
   (junction (at 176.53 101.6) (diameter 0) (color 0 0 0 0)
   )
+  (junction (at 128.27 71.12) (diameter 0) (color 0 0 0 0)
+  )
   (junction (at 45.72 43.18) (diameter 0) (color 0 0 0 0)
   )
@@
   (junction (at 132.08 101.6) (diameter 0) (color 0 0 0 0)
   )
+  (junction (at 138.43 71.12) (diameter 0) (color 0 0 0 0)
+  )
   (junction (at 69.85 90.17) (diameter 0) (color 0 0 0 0)
   )
@@
   (junction (at 54.61 60.96) (diameter 0) (color 0 0 0 0)
   )
+  (junction (at 80.01 71.12) (diameter 0) (color 0 0 0 0)
+  )
   (junction (at 45.72 50.8) (diameter 0) (color 0 0 0 0)
   )
@@
   )
   (junction (at 220.98 93.98) (diameter 0) (color 0 0 0 0)
+  )
+  (junction (at 104.14 71.12) (diameter 0) (color 0 0 0 0)
   )
   (junction (at 29.21 154.94) (diameter 0) (color 0 0 0 0)
@@
     (stroke (width 0) (type default))
   )
-  (wire (pts (xy 76.2 71.12) (xy 113.03 71.12))
+  (wire (pts (xy 76.2 71.12) (xy 80.01 71.12))
     (stroke (width 0) (type default))
   )
@@
     (stroke (width 0) (type default))
   )
+  (wire (pts (xy 128.27 71.12) (xy 138.43 71.12))
+    (stroke (width 0) (type default))
+  )
   (wire (pts (xy 71.12 156.21) (xy 69.85 156.21))
     (stroke (width 0) (type default))
@@
     (stroke (width 0) (type default))
   )
+  (wire (pts (xy 80.01 71.12) (xy 104.14 71.12))
+    (stroke (width 0) (type default))
+  )
   (wire (pts (xy 123.19 144.78) (xy 87.63 144.78))
     (stroke (width 0) (type default))
@@
     (stroke (width 0) (type default))
   )
+  (wire (pts (xy 138.43 71.12) (xy 147.32 71.12))
+    (stroke (width 0) (type default))
+  )
   (wire (pts (xy 118.11 95.25) (xy 127 95.25))
     (stroke (width 0) (type default))
@@
     (stroke (width 0) (type default))
   )
+  (wire (pts (xy 104.14 71.12) (xy 113.03 71.12))
+    (stroke (width 0) (type default))
+  )
   (wire (pts (xy 35.56 148.59) (xy 76.2 148.59))
     (stroke (width 0) (type default))
@@
     (stroke (width 0) (type default))
   )
-  (wire (pts (xy 113.03 71.12) (xy 147.32 71.12))
+  (wire (pts (xy 113.03 71.12) (xy 128.27 71.12))
     (stroke (width 0) (type default))
   )
@@
   (wire (pts (xy 176.53 50.8) (xy 176.53 13.97))
     (stroke (width 0) (type default))
+  )
+  (symbol (lib_id "Device:C") (at 104.14 74.93 0) (unit 1)
+    (in_bom yes) (on_board yes) (dnp no) (fields_autoplaced)
+    (property "Reference" "C74" (at 107.95 74.295 0)
+      (effects (font (size 1.27 1.27)) (justify left))
+    )
+    (property "Value" "10u" (at 107.95 76.835 0)
+      (effects (font (size 1.27 1.27)) (justify left))
+    )
+    (property "Footprint" "Capacitor_SMD:C_1210_3225Metric_Pad1.33x2.70mm_HandSolder" (at 105.1052 78.74 0)
+      (effects (font (size 1.27 1.27)) hide)
+    )
+    (property "Datasheet" "~" (at 104.14 74.93 0)
+      (effects (font (size 1.27 1.27)) hide)
+    )
+    (pin "1")
+    (pin "2")
+    (instances
+      (project "augertapowermanagement"
+        (path "/65134029-dbd2-409a-85a8-13c2a33ff019"
+          (reference "C74") (unit 1)
+        )
+      )
+    )
   )
   (symbol (lib_id "power:GND") (at 43.18 31.75 0) (unit 1)
@@
         (path "/65134029-dbd2-409a-85a8-13c2a33ff019"
           (reference "J2") (unit 1)
+        )
+      )
+    )
+  )
+  (symbol (lib_id "power:GND") (at 104.14 78.74 0) (unit 1)
+    (in_bom yes) (on_board yes) (dnp no)
+    (property "Reference" "#PWR067" (at 104.14 85.09 0)
+      (effects (font (size 1.27 1.27)) hide)
+    )
+    (property "Value" "GND" (at 107.95 77.47 0)
+      (effects (font (size 1.27 1.27)))
+    )
+    (property "Footprint" "" (at 104.14 78.74 0)
+      (effects (font (size 1.27 1.27)) hide)
+    )
+    (property "Datasheet" "" (at 104.14 78.74 0)
+      (effects (font (size 1.27 1.27)) hide)
+    )
+    (pin "1")
+    (instances
+      (project "augertapowermanagement"
+        (path "/65134029-dbd2-409a-85a8-13c2a33ff019"
+          (reference "#PWR067") (unit 1)
         )
       )
@@
         (path "/65134029-dbd2-409a-85a8-13c2a33ff019"
           (reference "J3") (unit 1)
+        )
+      )
+    )
+  )
+  (symbol (lib_id "power:GND") (at 80.01 78.74 0) (unit 1)
+    (in_bom yes) (on_board yes) (dnp no)
+    (property "Reference" "#PWR066" (at 80.01 85.09 0)
+      (effects (font (size 1.27 1.27)) hide)
+    )
+    (property "Value" "GND" (at 83.82 77.47 0)
+      (effects (font (size 1.27 1.27)))
+    )
+    (property "Footprint" "" (at 80.01 78.74 0)
+      (effects (font (size 1.27 1.27)) hide)
+    )
+    (property "Datasheet" "" (at 80.01 78.74 0)
+      (effects (font (size 1.27 1.27)) hide)
+    )
+    (pin "1")
+    (instances
+      (project "augertapowermanagement"
+        (path "/65134029-dbd2-409a-85a8-13c2a33ff019"
+          (reference "#PWR066") (unit 1)
         )
       )
@@
         (path "/65134029-dbd2-409a-85a8-13c2a33ff019"
           (reference "#PWR05") (unit 1)
+        )
+      )
+    )
+  )
+  (symbol (lib_id "Device:C") (at 128.27 74.93 0) (unit 1)
+    (in_bom yes) (on_board yes) (dnp no) (fields_autoplaced)
+    (property "Reference" "C71" (at 132.08 74.295 0)
+      (effects (font (size 1.27 1.27)) (justify left))
+    )
+    (property "Value" "10u" (at 132.08 76.835 0)
+      (effects (font (size 1.27 1.27)) (justify left))
+    )
+    (property "Footprint" "Capacitor_SMD:C_1210_3225Metric_Pad1.33x2.70mm_HandSolder" (at 129.2352 78.74 0)
+      (effects (font (size 1.27 1.27)) hide)
+    )
+    (property "Datasheet" "~" (at 128.27 74.93 0)
+      (effects (font (size 1.27 1.27)) hide)
+    )
+    (pin "1")
+    (pin "2")
+    (instances
+      (project "augertapowermanagement"
+        (path "/65134029-dbd2-409a-85a8-13c2a33ff019"
+          (reference "C71") (unit 1)
         )
       )
@@
     )
   )
+  (symbol (lib_id "Device:C") (at 80.01 74.93 0) (unit 1)
+    (in_bom yes) (on_board yes) (dnp no) (fields_autoplaced)
+    (property "Reference" "C73" (at 83.82 74.295 0)
+      (effects (font (size 1.27 1.27)) (justify left))
+    )
+    (property "Value" "10u" (at 83.82 76.835 0)
+      (effects (font (size 1.27 1.27)) (justify left))
+    )
+    (property "Footprint" "Capacitor_SMD:C_1210_3225Metric_Pad1.33x2.70mm_HandSolder" (at 80.9752 78.74 0)
+      (effects (font (size 1.27 1.27)) hide)
+    )
+    (property "Datasheet" "~" (at 80.01 74.93 0)
+      (effects (font (size 1.27 1.27)) hide)
+    )
+    (pin "1")
+    (pin "2")
+    (instances
+      (project "augertapowermanagement"
+        (path "/65134029-dbd2-409a-85a8-13c2a33ff019"
+          (reference "C73") (unit 1)
+        )
+      )
+    )
+  )
   (symbol (lib_id "Connector:TestPoint") (at 110.49 64.77 0) (unit 1)
     (in_bom yes) (on_board yes) (dnp no)
@@
     )
   )
+  (symbol (lib_id "power:GND") (at 128.27 78.74 0) (unit 1)
+    (in_bom yes) (on_board yes) (dnp no)
+    (property "Reference" "#PWR064" (at 128.27 85.09 0)
+      (effects (font (size 1.27 1.27)) hide)
+    )
+    (property "Value" "GND" (at 132.08 77.47 0)
+      (effects (font (size 1.27 1.27)))
+    )
+    (property "Footprint" "" (at 128.27 78.74 0)
+      (effects (font (size 1.27 1.27)) hide)
+    )
+    (property "Datasheet" "" (at 128.27 78.74 0)
+      (effects (font (size 1.27 1.27)) hide)
+    )
+    (pin "1")
+    (instances
+      (project "augertapowermanagement"
+        (path "/65134029-dbd2-409a-85a8-13c2a33ff019"
+          (reference "#PWR064") (unit 1)
+        )
+      )
+    )
+  )
   (symbol (lib_name "GND_2") (lib_id "power:GND") (at 22.86 60.96 0) (unit 1)
     (in_bom yes) (on_board yes) (dnp no) (fields_autoplaced)
@@
         (path "/65134029-dbd2-409a-85a8-13c2a33ff019"
           (reference "H4") (unit 1)
+        )
+      )
+    )
+  )
+  (symbol (lib_id "power:GND") (at 138.43 78.74 0) (unit 1)
+    (in_bom yes) (on_board yes) (dnp no)
+    (property "Reference" "#PWR065" (at 138.43 85.09 0)
+      (effects (font (size 1.27 1.27)) hide)
+    )
+    (property "Value" "GND" (at 142.24 77.47 0)
+      (effects (font (size 1.27 1.27)))
+    )
+    (property "Footprint" "" (at 138.43 78.74 0)
+      (effects (font (size 1.27 1.27)) hide)
+    )
+    (property "Datasheet" "" (at 138.43 78.74 0)
+      (effects (font (size 1.27 1.27)) hide)
+    )
+    (pin "1")
+    (instances
+      (project "augertapowermanagement"
+        (path "/65134029-dbd2-409a-85a8-13c2a33ff019"
+          (reference "#PWR065") (unit 1)
         )
       )
@@
         )
       )
+    )
+  )
+  (symbol (lib_id "Device:C") (at 138.43 74.93 0) (unit 1)
+    (in_bom yes) (on_board yes) (dnp no) (fields_autoplaced)
+    (property "Reference" "C72" (at 142.24 74.295 0)
+      (effects (font (size 1.27 1.27)) (justify left))
+    )
+    (property "Value" "10u" (at 142.24 76.835 0)
+      (effects (font (size 1.27 1.27)) (justify left))
+    )
+    (property "Footprint" "Capacitor_SMD:C_1210_3225Metric_Pad1.33x2.70mm_HandSolder" (at 139.3952 78.74 0)
+      (effects (font (size 1.27 1.27)) hide)
+    )
+    (property "Datasheet" "~" (at 138.43 74.93 0)
+      (effects (font (size 1.27 1.27)) hide)
+    )
+    (pin "1")
+    (pin "2")
+    (instances
+      (project "augertapowermanagement"
+        (path "/65134029-dbd2-409a-85a8-13c2a33ff019"
+          (reference "C72") (unit 1)
+        )
+      )

Commit message: update
Parts:
- C1: MANUFACTURER (none) -> B43547A9687M000; Purchase (none) -> https://www.digikey.com/en/products/detail/epcos-tdk-electr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
- C2: value 0.1 -> 0.1u X7R; MANUFACTURER (none) -> KGM32HR72D104KU; Purchase https://www.digikey.com/en/products/detail/kemet/CDR33BX104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 -> https://www.digikey.com/en/products/detail/kyocera-avx/KGM3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
- C59, C71, C72, C73, C74: MANUFACTURER (none) -> CL32A106KAULNNE; Purchase (none) -> https://www.digikey.com/en/products/detail/samsung-electro-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
- D1, D2: MANUFACTURER (none) -> 1N4007GP-TP
- H1, H2, H3, H4, H5, H6: Purchase (none) -> NP
- J1, J3: MANUFACTURER (none) -> TB007-508-05BE
- J10, J11, J12, J9: MANUFACTURER (none) -> 61400826021
- J2: value Image shown is a representation only. Exact specifications should be obtained from the product data sheet. -> Battery in; MANUFACTURER (none) -> TB009-508-02BE
- J4: value 0ZCF0200AF2C -> 42819-2214; MANUFACTURER Molex -> 42819-2214; Purchase https://www.digikey.com/en/products/detail/molex/0768250002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 -> https://www.mouser.com/ProductDetail/Molex/42819-2214?qs=c8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
- J5, J6, J7: MANUFACTURER (none) -> TB007-508-10BE
- J8: MANUFACTURER (none) -> TB007-508-08BE; Purchase https://www.digikey.com/en/products/detail/cui-devices/TB002V-500-08BE/10064083 -> https://www.digikey.com/en/products/detail/cui-devices/TB007-508-08BE/10064133?s=N4IgjCBcpgDA7AViqAxlAZgQwDYGcBTAGhAHsoBtEAJgA4wAWOEAXRIAcAXKEAZU4BOASwB2AcxABfEgFoGKEOkjZ8xEADcRmXIRLlIVeAGZ4SVh26QQUyZKA
- JP1, JP2: Purchase https://www.digikey.com/en/products/detail/keystone-electro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 -> DNP
- K1, K2: MANUFACTURER (none) -> T9AS5D12-12
- Q1: MANUFACTURER (none) -> 2N3904TFR; Purchase https://www.digikey.com/en/products/detail/stmicroelectroni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 -> https://www.mouser.com/ProductDetail/onsemi-Fairchild/2N390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
- R1, R2: MANUFACTURER (none) -> RNCP1206FTD1K00
- SW1: MANUFACTURER (none) -> OS102011MA1QN1
- TP1, TP2, TP3: Purchase JUST PAD -> NP
- U1: MANUFACTURER Espressif Systems -> ESP32-DevKitC-32D
- U2: Purchase IN LAB -> DNP
- U25: MANUFACTURER (none) -> MC7812CTG; Purchase (none) -> https://www.digikey.com/en/products/detail/onsemi/MC7812CTG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
