File: Adjustable Regulator.kicad_sch (KiCad schematic)
At the start: 5 parts, among them U20 LM2596S-ADJ

Commit message: hi
Parts:
- removed C1: 680uF, symbol Device:C
- removed C3: 220uF, symbol Device:C
- removed D3: 1N5821, Diode_THT:D_DO-201AD_P15.24mm_Horizontal, symbol Diode:1N5821
- removed L1: 33uH, symbol Device:L
- removed U20: LM2596S-ADJ, Package_TO_SOT_SMD:TO-263-5_TabPin3, symbol Regulator_Switching:LM2596S-ADJ
- added C23, C34, C45, C56: C, symbol Device:C
- added L11: L, symbol Device:L
- added R24, R46, R57: R_US, symbol Device:R_US
- added RV11: R_Potentiometer, symbol Device:R_Potentiometer
- added U22: LMR51450, symbol LMR514x0:LMR514x0
Connections:
- net GND: now also C23.2, C45.2, R24.2, R57.2, U22.13 (PGND), U22.8 (AGND)
- net V_in: now also C23.1, U22.10 (Vin), U22.11 (Vin), U22.12 (Vin), U22.9 (EN)
- net V_out: now also C56.1, L11.2, R46.1, RV11.2
- new net: C34.1, U22.4 (Boot)
- new net: C34.2, L11.1, U22.1 (SW), U22.2 (SW), U22.3 (SW)
- new net: R24.1, U22.6 (RT)
- new net: R57.1, RV11.1, U22.7 (FB)
- new net: C45.1, R46.2
- no-connect marks 0 -> 2

Commit message: finish assigning componets
Parts:
- removed C23: C, symbol Device:C
- added C47: 33u, Capacitor_SMD:C_1206_3216Metric_Pad1.33x1.80mm_HandSolder, symbol Device:C
- C44: renamed from C34; value C -> 0.1u X7R; footprint (none) -> Capacitor_SMD:C_1210_3225Metric_Pad1.33x2.70mm_HandSolder
- C45: value C -> 33p; footprint (none) -> Capacitor_SMD:C_1210_3225Metric_Pad1.33x2.70mm_HandSolder
- C46: renamed from C56; value C -> 33u; footprint (none) -> Capacitor_SMD:C_1206_3216Metric_Pad1.33x1.80mm_HandSolder
- L11: value L -> 5.6u; footprint (none) -> Inductor_SMD:L_Bourns_SRP1770TA_16.9x16.9mm
- R44: renamed from R24; value R_US -> 18.2k; footprint (none) -> Resistor_SMD:R_1206_3216Metric_Pad1.30x1.75mm_HandSolder
- R45: renamed from R57; value R_US -> 100k; footprint (none) -> Resistor_SMD:R_1206_3216Metric_Pad1.30x1.75mm_HandSolder
- R46: value R_US -> 1k; footprint (none) -> Resistor_SMD:R_1206_3216Metric_Pad1.30x1.75mm_HandSolder
- RV11: value R_Potentiometer -> 50k; footprint (none) -> Potentiometer_SMD:Potentiometer_Bourns_3314J_Vertical
- U24: renamed from U22; footprint (none) -> LMR51:WSON_SDRRR_TEX-M
Connections:
- net GND: now also C46.2, RV11.1, C47.2; no longer R45.2
- net V_out: now also R45.1, C47.1; no longer RV11.2
- new net: R45.2, RV11.2, U24.7 (FB)
Other:
- note added: "Set frequency to 500k Hz if R24 left open"
- moved on the sheet: R45, RV11

Commit message: fix lot of errors
Parts:
- added C51, C63: 4.7u X7R, Capacitor_SMD:C_1210_3225Metric_Pad1.33x2.70mm_HandSolder, symbol Device:C
- added R59: 18.2k, Resistor_SMD:R_1206_3216Metric_Pad1.30x1.75mm_HandSolder, symbol Device:R_US
- RV11: value 50k -> 2k
Connections:
- net GND: now also C51.2, C63.2, R59.2; no longer RV11.1
- net V_in: now also C51.1, C63.1
- new net: R59.1, RV11.1

Commit message: update
Parts:
- R59: value 18.2k -> 10k
- RV11: value 2k -> 25k
Changed lines of the file:
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@@
       (effects (font (size 1.27 1.27)) (justify left))
     )
-    (property "Value" "18.2k" (at 120.65 102.235 0)
+    (property "Value" "10k" (at 120.65 102.235 0)
       (effects (font (size 1.27 1.27)) (justify left))
     )
@@
       (effects (font (size 1.27 1.27)))
     )
-    (property "Value" "2k" (at 127 96.52 90)
-      (effects (font (size 1.27 1.27)))
-    )
+    (property "Value" "25k" (at 127 96.52 90)
+      (effects (font (size 1.27 1.27)))
+    )

Commit message: update
Parts:
- C44: MANUFACTURER (none) -> KGM32HR72D104KU; Purchase (none) -> https://www.digikey.com/en/products/detail/kyocera-avx/KGM3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
- C45: MANUFACTURER (none) -> 12102U330JAT2A; Purchase (none) -> https://www.mouser.com/ProductDetail/KYOCERA-AVX/12102U330J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
- C46, C47: MANUFACTURER (none) -> C3216X5R1E336M160AC; Purchase (none) -> https://www.digikey.com/en/products/detail/tdk-corporation/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
- C51, C63: MANUFACTURER (none) -> CL32B475KBUYNNE; Purchase (none) -> https://www.digikey.com/en/products/detail/samsung-electro-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
- L11: MANUFACTURER (none) -> SRP1770C-5R6M; Purchase (none) -> https://www.digikey.com/en/products/detail/bourns-inc/SRP17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
- R44: MANUFACTURER (none) -> RC1206FR-0718K2L; Purchase (none) -> https://www.digikey.com/en/products/detail/yageo/RC1206FR-0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
- R45: MANUFACTURER (none) -> RG3216P-1003-B-T1; Purchase (none) -> https://www.digikey.com/en/products/detail/susumu/RG3216P-1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
- R46: MANUFACTURER (none) -> RNCP1206FTD1K00; Purchase (none) -> https://www.digikey.com/en/products/detail/stackpole-electr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
- R59: MANUFACTURER (none) -> CRGP1206F1M0; Purchase (none) -> https://www.digikey.com/en/products/detail/te-connectivity-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
- RV11: MANUFACTURER (none) -> 3314J-1-253E; Purchase (none) -> https://www.digikey.com/en/products/detail/bourns-inc/3314J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
- U24: MANUFACTURER (none) -> LMR51450FNDRRR; Purchase (none) -> https://www.digikey.com/en/products/detail/texas-instrument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
Changed lines of the file:
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@@
+      (effects (font (size 1.27 1.27)) hide)
+    )
+    (property "Description" "CAP CER 0.1UF 200V X7R 1210" (at 106.68 74.93 0)
+      (effects (font (size 1.27 1.27)) hide)
+    )
+    (property "MANUFACTURER" "KGM32HR72D104KU" (at 106.68 74.93 0)
+      (effects (font (size 1.27 1.27)) hide)
+    )
+    (property "Purchase" "https://www.digikey.com/en/products/detail/kyocera-avx/KGM32HR72D104KU/1116341" (at 106.68 74.93 0)
       (effects (font (size 1.27 1.27)) hide)
     )
@@
       (effects (font (size 1.27 1.27)) hide)
     )
+    (property "Description" "CAP CER 33UF 25V X5R 1206" (at 152.4 85.09 0)
+      (effects (font (size 1.27 1.27)) hide)
+    )
+    (property "MANUFACTURER" "C3216X5R1E336M160AC" (at 152.4 85.09 0)
+      (effects (font (size 1.27 1.27)) hide)
+    )
+    (property "Purchase" "https://www.digikey.com/en/products/detail/tdk-corporation/C3216X5R1E336M160AC/2792259" (at 152.4 85.09 0)
+      (effects (font (size 1.27 1.27)) hide)
+    )
     (pin "1")
     (pin "2")
@@
       (effects (font (size 1.27 1.27)) hide)
     )
+    (property "Description" "RES 1M OHM 1% 1/2W 1206" (at 118.11 100.33 0)
+      (effects (font (size 1.27 1.27)) hide)
+    )
+    (property "MANUFACTURER" "CRGP1206F1M0" (at 118.11 100.33 0)
+      (effects (font (size 1.27 1.27)) hide)
+    )
+    (property "Purchase" "https://www.digikey.com/en/products/detail/te-connectivity-passive-product/CRGP1206F1M0/8577176" (at 118.11 100.33 0)
+      (effects (font (size 1.27 1.27)) hide)
+    )
     (pin "1")
     (pin "2")
@@
     )
     (property "Datasheet" "~" (at 142.24 85.09 0)
+      (effects (font (size 1.27 1.27)) hide)
+    )
+    (property "Description" "CAP CER 33UF 25V X5R 1206" (at 142.24 85.09 0)
+      (effects (font (size 1.27 1.27)) hide)
+    )
+    (property "MANUFACTURER" "C3216X5R1E336M160AC" (at 142.24 85.09 0)
+      (effects (font (size 1.27 1.27)) hide)
+    )
+    (property "Purchase" "https://www.digikey.com/en/products/detail/tdk-corporation/C3216X5R1E336M160AC/2792259" (at 142.24 85.09 0)
       (effects (font (size 1.27 1.27)) hide)
     )
@@
     )
     (property "Datasheet" "" (at 77.47 73.66 0)
+      (effects (font (size 1.27 1.27)) hide)
+    )
+    (property "Description" "IC REG BUCK ADJ 5A 12WSON" (at 77.47 73.66 0)
+      (effects (font (size 1.27 1.27)) hide)
+    )
+    (property "MANUFACTURER" "LMR51450FNDRRR" (at 77.47 73.66 0)
+      (effects (font (size 1.27 1.27)) hide)
+    )
+    (property "Purchase" "https://www.digikey.com/en/products/detail/texas-instruments/LMR51450FNDRRR/17394915" (at 77.47 73.66 0)
       (effects (font (size 1.27 1.27)) hide)
     )
@@
       (effects (font (size 1.27 1.27)) hide)
     )
+    (property "Description" "FIXED IND 5.6UH 24A 6.8 MOHM SMD" (at 115.57 81.28 0)
+      (effects (font (size 1.27 1.27)) hide)
+    )
+    (property "MANUFACTURER" "SRP1770C-5R6M" (at 115.57 81.28 0)
+      (effects (font (size 1.27 1.27)) hide)
+    )
+    (property "Purchase" "https://www.digikey.com/en/products/detail/bourns-inc/SRP1770C-5R6M/10249071" (at 115.57 81.28 0)
+      (effects (font (size 1.27 1.27)) hide)
+    )
     (pin "1")
     (pin "2")
@@
     )
     (property "Datasheet" "~" (at 132.08 92.71 0)
+      (effects (font (size 1.27 1.27)) hide)
+    )
+    (property "Description" "Multilayer Ceramic Capacitors MLCC - SMD/SMT 200V 33 pF 0.05 ULTRA LOW ESR" (at 132.08 92.71 0)
+      (effects (font (size 1.27 1.27)) hide)
+    )
+    (property "MANUFACTURER" "12102U330JAT2A" (at 132.08 92.71 0)
+      (effects (font (size 1.27 1.27)) hide)
+    )
+    (property "Purchase" "https://www.mouser.com/ProductDetail/KYOCERA-AVX/12102U330JAT2A?qs=Si5KMF%252BzaWIH9qeLgPv8dg%3D%3D" (at 132.08 92.71 0)
       (effects (font (size 1.27 1.27)) hide)
     )
@@
       (effects (font (size 1.27 1.27)) hide)
     )
+    (property "Description" "TRIMMER 25K OHM 0.25W J LEAD TOP" (at 121.92 92.71 0)
+      (effects (font (size 1.27 1.27)) hide)
+    )
+    (property "MANUFACTURER" "3314J-1-253E" (at 121.92 92.71 0)
+      (effects (font (size 1.27 1.27)) hide)
+    )
+    (property "Purchase" "https://www.digikey.com/en/products/detail/bourns-inc/3314J-1-253E/86643" (at 121.92 92.71 0)
+      (effects (font (size 1.27 1.27)) hide)
+    )
     (pin "1")
     (pin "2")
@@
       (effects (font (size 1.27 1.27)) hide)
     )
+    (property "Description" "CAP CER 4.7UF 50V X7R 1210" (at 50.8 77.47 0)
+      (effects (font (size 1.27 1.27)) hide)
+    )
+    (property "MANUFACTURER" "CL32B475KBUYNNE" (at 50.8 77.47 0)
+      (effects (font (size 1.27 1.27)) hide)
+    )
+    (property "Purchase" "https://www.digikey.com/en/products/detail/samsung-electro-mechanics/CL32B475KBUYNNE/3886950" (at 50.8 77.47 0)
+      (effects (font (size 1.27 1.27)) hide)
+    )
     (pin "1")
     (pin "2")
@@
       (effects (font (size 1.27 1.27)) hide)
     )
+    (property "Description" "RES 1K OHM 1% 1/2W 1206" (at 132.08 85.09 0)
+      (effects (font (size 1.27 1.27)) hide)
+    )
+    (property "MANUFACTURER" "RNCP1206FTD1K00" (at 132.08 85.09 0)
+      (effects (font (size 1.27 1.27)) hide)
+    )
+    (property "Purchase" "https://www.digikey.com/en/products/detail/stackpole-electronics-inc/RNCP1206FTD1K00/2240337" (at 132.08 85.09 0)
+      (effects (font (size 1.27 1.27)) hide)
+    )
     (pin "1")
     (pin "2")
@@
       (effects (font (size 1.27 1.27)) hide)
     )
+    (property "Description" "RES SMD 100K OHM 0.1% 1/4W 1206" (at 121.92 85.09 0)
+      (effects (font (size 1.27 1.27)) hide)
+    )
+    (property "MANUFACTURER" "RG3216P-1003-B-T1" (at 121.92 85.09 0)
+      (effects (font (size 1.27 1.27)) hide)
+    )
+    (property "Purchase" "https://www.digikey.com/en/products/detail/susumu/RG3216P-1003-B-T1/1272606" (at 121.92 85.09 0)
+      (effects (font (size 1.27 1.27)) hide)
+    )
     (pin "1")
     (pin "2")
@@
       (effects (font (size 1.27 1.27)) hide)
     )
+    (property "Description" "CAP CER 4.7UF 50V X7R 1210" (at 64.77 76.2 0)
+      (effects (font (size 1.27 1.27)) hide)
+    )
+    (property "MANUFACTURER" "CL32B475KBUYNNE" (at 64.77 76.2 0)
+      (effects (font (size 1.27 1.27)) hide)
+    )
+    (property "Purchase" "https://www.digikey.com/en/products/detail/samsung-electro-mechanics/CL32B475KBUYNNE/3886950" (at 64.77 76.2 0)
+      (effects (font (size 1.27 1.27)) hide)
+    )
     (pin "1")
     (pin "2")
@@
       (effects (font (size 1.27 1.27)) hide)
     )
+    (property "Description" "RES 18.2K OHM 1% 1/4W 1206" (at 54.61 93.98 0)
+      (effects (font (size 1.27 1.27)) hide)
+    )
+    (property "MANUFACTURER" "RC1206FR-0718K2L" (at 54.61 93.98 0)
+      (effects (font (size 1.27 1.27)) hide)
+    )
+    (property "Purchase" "https://www.digikey.com/en/products/detail/yageo/RC1206FR-0718K2L/728594" (at 54.61 93.98 0)
+      (effects (font (size 1.27 1.27)) hide)
+    )
